File: KiCAD PCB Files/P4-Audio-TFT/P4-Audio-TFT.kicad_pcb (KiCad board)
At the start: 4 copper layers, 108 x 60.9 mm, 188 parts, among them J1 USB-C Program, J2 Headphone, J3 Type B Host, J4 Line-Out, J5 EXPANSION, J6 Micro_SD_Card, J7 C6 PROG, Q1 EMH4T2R, Q2 AO3401A, Q3 AO3400A, SW1 Card Detect, SW2 RESET, SW3 POWER, U1 CH340C, U2 PCM5102, U3 ES8388, U4 ESP32-P4NRW32X, U5 TLV62569DBV, U6 W25Q256JVEIQ, U7 TLV62569DBV, U8 TPS61183RTJT, U9 ESP32-C6-MINI-1/U, Y1 40Mhz, Y2 32.768Khz

Commit message: 2nd PCB edit
Parts:
- moved U7 30.8 mm to (104.6, 89.5)
- moved SW1 24.2 mm to (139.2, 79.4), turned to 0 degrees
- moved U1 12.4 mm to (74.4, 74.3), turned to 90 degrees
- moved U5 12.1 mm to (104.6, 78.5)
- moved Q1 9.03 mm to (74.3, 84.6), turned to 180 degrees
- moved U2 7.78 mm to (127.2, 81.3)
- moved U3 5.69 mm to (133.3, 96.2)
- moved U9 0.73 mm to (75.3, 108.7)
Other:
- outline, holes or cut-outs redrawn

Commit message: PCB WS and P4-C6 complete
Parts:
- removed C62, C64, C71: 10uF, Capacitor_SMD:C_0603_1608Metric
- removed C63: 6.8pF, Capacitor_SMD:C_0603_1608Metric
- removed C69, C70: 0.1uF, Capacitor_SMD:C_0603_1608Metric
- removed the C76 at (-174.4, -50.6)
- removed the C76 at (-68.3, -85.0)
- removed the C77 at (-43.8, -81.4)
- removed the C77 at (-174.4, -43.6)
- removed C8: 30PF, Capacitor_SMD:C_0603_1608Metric
- removed C83, C84: 100uF, Capacitor_SMD:CP_Elec_6.3x5.8
- removed J4: Line-Out, Connector_Audio:Jack_3.5mm_PJ320D_Horizontal
- removed L3: 2.2uH, Inductor_SMD:L_0805_2012Metric
- removed Q1: EMH4T2R, Package_TO_SOT_SMD:SOT-563
- removed the R10 at (-304.3, -114.1)
- removed the R10 at (-312.5, -158.6)
- removed the R11 at (-312.9, -150.2)
- removed the R11 at (-303.6, -108.3)
- removed the R12 at (-303.6, -101.5)
- removed the R12 at (-305.5, -150.1)
- removed the R13 at (-302.3, -94.8)
- removed the R13 at (-313.1, -142.0)
- removed the R14 at (-278.9, -168.8)
- removed the R14 at (-274.4, -115.9)
- removed the R15 at (-297.0, -168.7)
- removed the R15 at (-273.3, -107.9)
- removed the R15 at (-287.0, -81.6)
- removed the R16 at (-304.1, -160.4)
- removed the R16 at (-309.7, -106.3)
- removed R20: 100K, Resistor_SMD:R_0603_1608Metric
- removed R21: 22K1, Resistor_SMD:R_0603_1608Metric
- removed R22: 200K, Resistor_SMD:R_0603_1608Metric
- removed the R23 at (-297.4, -152.6)
- removed the R23 at (-287.6, -75.8)
- removed the R24 at (-297.2, -143.2)
- removed the R24 at (-275.3, -100.7)
- removed the R25 at (-289.3, -169.6)
- removed the R25 at (-259.9, -96.2)
- removed the R27 at (-287.2, -163.2)
- removed the R27 at (-298.3, -121.4)
- removed R28 (x2), R39: 10K, Resistor_SMD:R_0603_1608Metric
- removed the R29 at (-289.4, -146.1)
- removed the R29 at (-283.6, -121.5)
- removed the R30 at (-296.9, -108.9)
- removed the R30 at (-295.7, -132.2)
- removed the R31 at (-305.3, -133.7)
- removed the R31 at (-296.0, -102.2)
- removed the R32 at (-289.4, -100.9)
- removed the R32 at (-312.9, -133.0)
- removed the R33 at (-277.2, -160.9)
- removed the R33 at (-296.0, -95.9)
- removed the R34 at (-275.5, -154.9)
- removed the R34 at (-288.0, -95.9)
- removed the R35 at (-281.0, -96.0)
- removed the R35 at (-250.8, -67.0)
- removed R41, R42, R45: 51K, Resistor_SMD:R_0603_1608Metric
- removed the R6 at (-332.4, -101.9)
- removed the R6 at (-265.1, -101.7)
- removed the R7 at (-271.2, -96.4)
- removed the R7 at (-303.3, -167.9)
- removed the U1 at (74.4, 74.3)
- removed U7: TLV62569DBV, Package_TO_SOT_SMD:SOT-23-5
- added BT1: BS-12-B3AA011, P4Local_Coin_Cell:MYOUNG_BS-12-B3AA011_C964729, B.Cu at (100.3, 131.5)
- added C136: 100nF, P4Local_Capacitor_SMD:C_0603_1608Metric, B.Cu at (85.0, 69.8)
- added C137: 100nF, P4Local_Capacitor_SMD:C_0603_1608Metric, B.Cu at (90.5, 77.5)
- added C138: 10uF, P4Local_Capacitor_SMD:C_0805_2012Metric, B.Cu at (94.0, 77.5)
- added C17: 100nF, P4Local_Capacitor_SMD:C_0603_1608Metric, B.Cu at (132.1, 90.5)
- added C18: 100nF, P4Local_Capacitor_SMD:C_0603_1608Metric, B.Cu at (86.0, 77.3)
- added C23: 100nF, P4Local_Capacitor_SMD:C_0603_1608Metric, B.Cu at (113.8, 99.8)
- added C29: 100nF, P4Local_Capacitor_SMD:C_0603_1608Metric, B.Cu at (112.9, 106.3)
- added C30: 100nF, P4Local_Capacitor_SMD:C_0603_1608Metric, B.Cu at (103.3, 100.1)
- added C31: 10uF, P4Local_Capacitor_SMD:C_0603_1608Metric, B.Cu at (148.4, 129.0)
- added C32: 10uF, P4Local_Capacitor_SMD:C_0603_1608Metric, B.Cu at (122.7, 94.7)
- added C33: 100nF, P4Local_Capacitor_SMD:C_0603_1608Metric, B.Cu at (122.7, 93.0)
- added C34: 100nF, P4Local_Capacitor_SMD:C_0603_1608Metric, B.Cu at (132.1, 92.2)
- added C65: 100nF, P4Local_Capacitor_SMD:C_0603_1608Metric, B.Cu at (97.0, 74.2)
- added C66: 10uF, P4Local_Capacitor_SMD:C_0805_2012Metric, B.Cu at (93.2, 84.3)
- added C76: 10uF, P4Local_Capacitor_SMD:C_0603_1608Metric, B.Cu at (69.4, 136.3)
- added C77: 100nF, P4Local_Capacitor_SMD:C_0603_1608Metric, B.Cu at (69.4, 134.2)
- added C81: 10uF, P4Local_Capacitor_SMD:C_0805_2012Metric, B.Cu at (93.2, 79.7)
- added C82: 100nF, P4Local_Capacitor_SMD:C_0603_1608Metric, B.Cu at (82.8, 74.9)
- added C85: 100nF, P4Local_Capacitor_SMD:C_0603_1608Metric, B.Cu at (74.5, 84.5)
- added C86: 100nF, P4Local_Capacitor_SMD:C_0603_1608Metric, B.Cu at (77.8, 134.4)
- added C87: 1uF, P4Local_Capacitor_SMD:C_0603_1608Metric, B.Cu at (96.0, 119.9)
- added C88: 22uF, P4Local_Capacitor_SMD:C_0805_2012Metric, B.Cu at (98.4, 119.9)
- added C89: 2.2uF, P4Local_Capacitor_SMD:C_0603_1608Metric, B.Cu at (138.0, 88.5)
- added C90: 1uF, P4Local_Capacitor_SMD:C_0603_1608Metric, B.Cu at (135.0, 94.5)
- added C91: 1uF, P4Local_Capacitor_SMD:C_0603_1608Metric, B.Cu at (135.0, 97.0)
- added C92: 100pF, P4Local_Capacitor_SMD:C_0603_1608Metric, B.Cu at (138.5, 94.5)
- added C93: 100pF, P4Local_Capacitor_SMD:C_0603_1608Metric, B.Cu at (138.5, 97.0)
- added J10: S7B-PH-SM4-TB(LF)(SN), P4Local_Connector_JST:JST_PH_S7B-PH-SM4-TB_1x07-1MP_P2.00mm_Horizontal, B.Cu at (93.0, 145.0)
- added J11: S8B-PH-SM4-TB(LF)(SN), P4Local_Connector_JST:JST_PH_S8B-PH-SM4-TB_1x08-1MP_P2.00mm_Horizontal, B.Cu at (115.0, 145.0)
- added J12: S5B-PH-SM4-TB(LF)(SN), P4Local_Connector_JST:JST_PH_S5B-PH-SM4-TB_1x05-1MP_P2.00mm_Horizontal, B.Cu at (55.0, 116.0)
- added J13: S5B-PH-SM4-TB(LF)(SN), P4Local_Connector_JST:JST_PH_S5B-PH-SM4-TB_1x05-1MP_P2.00mm_Horizontal, B.Cu at (55.0, 89.0)
- added J8: VBAT_SELECT, P4Local_Connector_JST:PinHeader_1x03_P2.54mm_Horizontal, F.Cu at (61.0, 79.5)
- added J9: S5B-PH-SM4-TB(LF)(SN), P4Local_Connector_JST:JST_PH_S5B-PH-SM4-TB_1x05-1MP_P2.00mm_Horizontal, B.Cu at (75.0, 145.0)
- added Q4: S8050, P4Core:SOT-23, B.Cu at (75.0, 88.5)
- added Q5: S8050, P4Core:SOT-23, B.Cu at (80.0, 88.5)
- added R10: 22R, P4Local_Resistor_SMD:R_0603_1608Metric, B.Cu at (123.0, 97.1)
- added R11: 22R, P4Local_Resistor_SMD:R_0603_1608Metric, B.Cu at (124.6, 97.1)
- added R12: 10k, P4Local_Resistor_SMD:R_0603_1608Metric, B.Cu at (102.2, 104.5)
- added R13: 470R, P4Local_Resistor_SMD:R_0603_1608Metric, B.Cu at (117.5, 104.8)
- added R14: 470R, P4Local_Resistor_SMD:R_0603_1608Metric, B.Cu at (117.5, 107.0)
- added R15: 100R, P4Local_Resistor_SMD:R_0603_1608Metric, B.Cu at (100.5, 112.9)
- added R16: 5.1k, P4Local_Resistor_SMD:R_0603_1608Metric, B.Cu at (94.2, 71.0)
- added R18: 10k, P4Local_Resistor_SMD:R_0603_1608Metric, B.Cu at (145.0, 142.0)
- added R23: 100k, P4Local_Resistor_SMD:R_0603_1608Metric, B.Cu at (100.5, 109.7)
- added R24: 5.1k, P4Local_Resistor_SMD:R_0603_1608Metric, B.Cu at (79.5, 75.0)
- added R25: 10k, P4Local_Resistor_SMD:R_0603_1608Metric, B.Cu at (137.8, 108.5)
- added R27: 5.1k, P4Local_Resistor_SMD:R_0603_1608Metric, B.Cu at (75.7, 75.0)
- added R29: 10k, P4Local_Resistor_SMD:R_0603_1608Metric, B.Cu at (116.0, 121.8)
- added R30: 10k, P4Local_Resistor_SMD:R_0603_1608Metric, B.Cu at (71.0, 131.0)
- added R31: 10k, P4Local_Resistor_SMD:R_0603_1608Metric, B.Cu at (74.3, 131.0)
- added R32: 10k, P4Local_Resistor_SMD:R_0603_1608Metric, B.Cu at (72.5, 133.0)
- added R33: 10k, P4Local_Resistor_SMD:R_0603_1608Metric, B.Cu at (74.0, 135.2)
- added R34: 10k, P4Local_Resistor_SMD:R_0603_1608Metric, B.Cu at (74.0, 137.5)
- added R35: 10k, P4Local_Resistor_SMD:R_0603_1608Metric, B.Cu at (54.8, 144.3)
- added R47: 1k, P4Local_Resistor_SMD:R_0603_1608Metric, B.Cu at (138.0, 86.5)
- added R48: 2k, P4Local_Resistor_SMD:R_0603_1608Metric, B.Cu at (138.0, 90.5)
- added R6: 33R, P4Local_Resistor_SMD:R_0603_1608Metric, B.Cu at (116.0, 130.2)
- added R60: 60.4k, P4Local_Resistor_SMD:R_0603_1608Metric, B.Cu at (91.5, 72.5)
- added R61: 10k, P4Local_Resistor_SMD:R_0603_1608Metric, B.Cu at (75.0, 91.5)
- added R62: 10k, P4Local_Resistor_SMD:R_0603_1608Metric, B.Cu at (80.0, 91.5)
- added R7: 33R, P4Local_Resistor_SMD:R_0603_1608Metric, B.Cu at (116.0, 134.4)
- added U10: TPS2553DBVR, P4Core:SOT-23-6, B.Cu at (87.5, 72.5)
- added U4: CH340C, P4Local_Package_SO:SOIC-16_3.9x9.9mm_P1.27mm, B.Cu at (79.9, 79.6)
- C1, C2, C24, C26, C27, C28, C4, C75: footprint Capacitor_SMD:C_0603_1608Metric -> P4Local_Capacitor_SMD:C_0603_1608Metric; moved to B.Cu
- C10, C12: value 4.7uF -> 100nF; footprint Capacitor_SMD:C_0603_1608Metric -> P4Local_Capacitor_SMD:C_0603_1608Metric; moved to B.Cu
- C100: renamed from C34; footprint Capacitor_SMD:C_0603_1608Metric -> P4Core:C_0603_1608Metric; moved to B.Cu
- C101: renamed from C35; value 0.1uF -> 100nF; footprint Capacitor_SMD:C_0603_1608Metric -> P4Core:C_0402_1005Metric; moved to B.Cu
- C102: renamed from C36; footprint Capacitor_SMD:C_0603_1608Metric -> P4Core:C_0402_1005Metric; moved to B.Cu
- C103: renamed from C37; value 0.1uF -> 100nF; footprint Capacitor_SMD:C_0603_1608Metric -> P4Core:C_0603_1608Metric; moved to B.Cu
- C104: renamed from C38; value 0.1uF -> 100nF; footprint Capacitor_SMD:C_0603_1608Metric -> P4Core:C_0603_1608Metric; moved to B.Cu
- C105: renamed from C39; value 0.1uF -> 100nF; footprint Capacitor_SMD:C_0603_1608Metric -> P4Core:C_0603_1608Metric; moved to B.Cu
- C106: renamed from C40; footprint Capacitor_SMD:C_0603_1608Metric -> P4Core:C_0603_1608Metric; moved to B.Cu
- C107: renamed from C41; value 0.1uF -> 100nF; footprint Capacitor_SMD:C_0603_1608Metric -> P4Core:C_0603_1608Metric; moved to B.Cu
- C108: renamed from C42; footprint Capacitor_SMD:C_0603_1608Metric -> P4Core:C_0603_1608Metric; moved to B.Cu
- C109: renamed from C43; value 0.1uF -> 100nF; footprint Capacitor_SMD:C_0603_1608Metric -> P4Core:C_0603_1608Metric; moved to B.Cu
- C11, C13, C15, C21, C9: value 0.1uF -> 10uF; footprint Capacitor_SMD:C_0603_1608Metric -> P4Local_Capacitor_SMD:C_0603_1608Metric; moved to B.Cu
- C110: renamed from C44; value 0.1uF -> 100nF; footprint Capacitor_SMD:C_0603_1608Metric -> P4Core:C_0603_1608Metric; moved to B.Cu
- C111: renamed from C45; footprint Capacitor_SMD:C_0603_1608Metric -> P4Core:C_0603_1608Metric; moved to B.Cu
- C112: renamed from C46; value 0.1uF -> 100nF; footprint Capacitor_SMD:C_0603_1608Metric -> P4Core:C_0603_1608Metric; moved to B.Cu
- C113: renamed from C47; footprint Capacitor_SMD:C_0603_1608Metric -> P4Core:C_0603_1608Metric; moved to B.Cu
- C114: renamed from C48; value 0.1uF -> 100nF; footprint Capacitor_SMD:C_0603_1608Metric -> P4Core:C_0603_1608Metric; moved to B.Cu
- C115: renamed from C49; value 0.1uF -> 100nF; footprint Capacitor_SMD:C_0603_1608Metric -> P4Core:C_0402_1005Metric; moved to B.Cu
- C116: renamed from C50; footprint Capacitor_SMD:C_0603_1608Metric -> P4Core:C_0402_1005Metric; moved to B.Cu
- C117: renamed from C51; value 0.1uF -> 100nF; footprint Capacitor_SMD:C_0603_1608Metric -> P4Core:C_0603_1608Metric; moved to B.Cu
- C118: renamed from C52; value 0.1uF -> 100nF; footprint Capacitor_SMD:C_0603_1608Metric -> P4Core:C_0402_1005Metric; moved to B.Cu
- C119: renamed from C53; footprint Capacitor_SMD:C_0603_1608Metric -> P4Core:C_0603_1608Metric; moved to B.Cu
- C120: renamed from C54; footprint Capacitor_SMD:C_0603_1608Metric -> P4Core:C_0603_1608Metric; moved to B.Cu
- C121: renamed from C55; footprint Capacitor_SMD:C_0603_1608Metric -> P4Core:C_0603_1608Metric; moved to B.Cu
- C122: renamed from C56; footprint Capacitor_SMD:C_0603_1608Metric -> P4Core:C_0603_1608Metric; moved to B.Cu
- C123: renamed from C57; footprint Capacitor_SMD:C_0603_1608Metric -> P4Core:C_0603_1608Metric; moved to B.Cu
- C124: renamed from C58; footprint Capacitor_SMD:C_0603_1608Metric -> P4Core:C_0603_1608Metric; moved to B.Cu
- C125: renamed from C59; footprint Capacitor_SMD:C_0603_1608Metric -> P4Core:C_0603_1608Metric; moved to B.Cu
- C126: renamed from C60; footprint Capacitor_SMD:C_0603_1608Metric -> P4Core:C_0603_1608Metric; moved to B.Cu
- C127: renamed from C61; value 0.1uF -> 100nF; footprint Capacitor_SMD:C_0603_1608Metric -> P4Core:C_0603_1608Metric; moved to B.Cu
- C128: renamed from C67; footprint Capacitor_SMD:C_0603_1608Metric -> P4Core:C_0603_1608Metric; moved to B.Cu
- C129: renamed from C68; value 0.1uF -> 100nF; footprint Capacitor_SMD:C_0603_1608Metric -> P4Core:C_0603_1608Metric; moved to B.Cu
- C130: renamed from C72; footprint Capacitor_SMD:C_0603_1608Metric -> P4Core:C_0603_1608Metric; moved to B.Cu
- C131: renamed from C73; value 0.1uF -> 100nF; footprint Capacitor_SMD:C_0603_1608Metric -> P4Core:C_0603_1608Metric; moved to B.Cu
- C132: renamed from C74; value 0.1uF -> 100nF; footprint Capacitor_SMD:C_0603_1608Metric -> P4Core:C_0603_1608Metric; moved to B.Cu
- C133: renamed from C78; value 0.1uF -> 100nF; footprint Capacitor_SMD:C_0603_1608Metric -> P4Core:C_0603_1608Metric; moved to B.Cu
- C134: renamed from C79; footprint Capacitor_SMD:C_0603_1608Metric -> P4Core:C_0603_1608Metric; moved to B.Cu
- C135: renamed from C80; footprint Capacitor_SMD:C_0603_1608Metric -> P4Core:C_0603_1608Metric; moved to B.Cu
- C14, C16, C22: value 10uF -> 100nF; footprint Capacitor_SMD:C_0603_1608Metric -> P4Local_Capacitor_SMD:C_0603_1608Metric; moved to B.Cu
- C19, C25, C5, C6: value 0.1uF -> 100nF; footprint Capacitor_SMD:C_0603_1608Metric -> P4Local_Capacitor_SMD:C_0603_1608Metric; moved to B.Cu
- C20: value 0.1uF -> 22uF; footprint Capacitor_SMD:C_0603_1608Metric -> P4Local_Capacitor_SMD:C_0805_2012Metric; moved to B.Cu
- C3: value 30pF -> 100uF; footprint Capacitor_SMD:C_0603_1608Metric -> P4Local_Capacitor_SMD:C_1206_3216Metric; moved to B.Cu
- C7: value 30PF -> 100uF; footprint Capacitor_SMD:C_0603_1608Metric -> P4Local_Capacitor_SMD:C_1206_3216Metric; moved to B.Cu
- C94: renamed from C23; value 0.1uF -> 100nF; footprint Capacitor_SMD:C_0603_1608Metric -> P4Core:C_0603_1608Metric; moved to B.Cu
- C95: renamed from C29; value 0.1uF -> 100nF; footprint Capacitor_SMD:C_0603_1608Metric -> P4Core:C_0603_1608Metric; moved to B.Cu
- C96: renamed from C30; value 0.1uF -> 100nF; footprint Capacitor_SMD:C_0603_1608Metric -> P4Core:C_0603_1608Metric; moved to B.Cu
- C97: renamed from C31; footprint Capacitor_SMD:C_0603_1608Metric -> P4Core:C_0603_1608Metric; moved to B.Cu
- C98: renamed from C32; footprint Capacitor_SMD:C_0603_1608Metric -> P4Core:C_0603_1608Metric; moved to B.Cu
- C99: renamed from C33; footprint Capacitor_SMD:C_0603_1608Metric -> P4Core:C_0402_1005Metric; moved to B.Cu
- D1: value LED -> Green LED; footprint LED_SMD:LED_0603_1608Metric -> P4Local_LED_SMD:LED_0805_2012Metric; moved to B.Cu
- D3: value SS36 -> SS34; footprint Diode_SMD:D_SMA -> P4Local_Diode_SMD:D_SMA; moved to B.Cu
- DS1: value ILI TFT Panel -> FH34SRJ-40S-0.5SH(50); footprint ILI9488_TFT_40P:ILI9488_TFT_40P_ALIGNED_V3 -> P4Local_Updated:ILI9488_40P_4inch_Checked; moved to B.Cu
- H1, H2, H3, H4: value ~ -> MountingHole; footprint MountingHole:MountingHole_3.2mm_M3 -> P4Local_MountingHole:MountingHole_3.2mm_M3
- J1: value USB-C Program -> TYPE-C-31-M-12; footprint Connector_USB:USB_C_Receptacle_HRO_TYPE-C-31-M-12 -> P4Local_Connector_USB:USB_C_Receptacle_HRO_TYPE-C-31-M-12
- J2: value Headphone -> PJ-320D; footprint Connector_Audio:Jack_3.5mm_PJ320D_Horizontal -> P4Local_Connector_Audio_Han:HanElectricity_PJ320D_C22459515
- J3: value Type B Host -> PJ-320D; footprint Connector_USB:USB_A_Molex_67643_Horizontal -> P4Local_Connector_Audio_Han:HanElectricity_PJ320D_C22459515
- J5: value EXPANSION -> 67643-3911; footprint Connector_PinSocket_2.54mm:PinSocket_2x10_P2.54mm_Vertical -> P4Local_Connector_USB:USB_A_Molex_67643_Horizontal
- J6: value Micro_SD_Card -> DM3AT-SF-PEJM5; footprint Connector_Card:microSD_HC_Hirose_DM3AT-SF-PEJM5 -> P4Local_Connector_Card:microSD_HC_Hirose_DM3AT-SF-PEJM5; moved to B.Cu
- J7: value C6 PROG -> Conn_01x04_Pin; footprint Connector_PinHeader_2.54mm:PinHeader_1x04_P2.54mm_Vertical -> P4Local_Connector_PinHeader_2_54mm:PinHeader_1x04_P2.54mm_Vertical
- L1: value 600R@100Mhz -> 600R@100MHz Ferrite; footprint Inductor_SMD:L_0603_1608Metric -> P4Local_Inductor_SMD:L_0603_1608Metric; moved to B.Cu
- L2: value 1uH 2.5*2*1.2 3.5A -> 1uH; footprint Inductor_SMD:L_0805_2012Metric -> P4Core:L_INMICRO_IMTF201610; moved to B.Cu
- Q2, Q3: footprint Package_TO_SOT_SMD:SOT-23 -> P4Local_Package_TO_SOT_SMD:SOT-23; moved to B.Cu
- R1, R2: value 1K -> 4.7k; footprint Resistor_SMD:R_0603_1608Metric -> P4Local_Resistor_SMD:R_0603_1608Metric; moved to B.Cu
- R17: value 200K -> 33R; footprint Resistor_SMD:R_0603_1608Metric -> P4Local_Resistor_SMD:R_0603_1608Metric; moved to B.Cu
- R26: value 16R -> 16R 0.5W; footprint Resistor_SMD:R_1206_3216Metric -> P4Local_Resistor_SMD:R_1210_3225Metric; moved to B.Cu
- R3: value 330 -> 10k; footprint Resistor_SMD:R_0603_1608Metric -> P4Local_Resistor_SMD:R_0603_1608Metric; moved to B.Cu
- R36, R46: value 10K -> 10k; footprint Resistor_SMD:R_0603_1608Metric -> P4Local_Resistor_SMD:R_0603_1608Metric; moved to B.Cu
- R37: value 10K -> 100k; footprint Resistor_SMD:R_0603_1608Metric -> P4Local_Resistor_SMD:R_0603_1608Metric; moved to B.Cu
- R4: value 330 -> 10R; footprint Resistor_SMD:R_0603_1608Metric -> P4Local_Resistor_SMD:R_0603_1608Metric; moved to B.Cu
- R49: renamed from R17; value 200K -> 499k; footprint Resistor_SMD:R_0603_1608Metric -> P4Core:R_0603_1608Metric; moved to B.Cu
- R5, R8: footprint Resistor_SMD:R_0603_1608Metric -> P4Local_Resistor_SMD:R_0603_1608Metric; moved to B.Cu
- R50: renamed from R22; value 200K -> 499k; footprint Resistor_SMD:R_0603_1608Metric -> P4Core:R_0603_1608Metric; moved to B.Cu
- R51: renamed from R18; footprint Resistor_SMD:R_0603_1608Metric -> P4Core:R_0603_1608Metric; moved to B.Cu
- R52: renamed from R19; value 10K -> 10k; footprint Resistor_SMD:R_0603_1608Metric -> P4Core:R_0603_1608Metric; moved to B.Cu
- R53: renamed from R38; value 10K -> 10k; footprint Resistor_SMD:R_0603_1608Metric -> P4Core:R_0603_1608Metric; moved to B.Cu
- R54: renamed from R40; value 51K -> 51k; footprint Resistor_SMD:R_0603_1608Metric -> P4Core:R_0603_1608Metric; moved to B.Cu
- R55: renamed from R41; value 51K -> 51k; footprint Resistor_SMD:R_0603_1608Metric -> P4Core:R_0603_1608Metric; moved to B.Cu
- R56: renamed from R42; value 51K -> 51k; footprint Resistor_SMD:R_0603_1608Metric -> P4Core:R_0603_1608Metric; moved to B.Cu
- R57: renamed from R43; value 51K -> 51k; footprint Resistor_SMD:R_0603_1608Metric -> P4Core:R_0603_1608Metric; moved to B.Cu
- R58: renamed from R44; value 51K -> 51k; footprint Resistor_SMD:R_0603_1608Metric -> P4Core:R_0603_1608Metric; moved to B.Cu
- R59: renamed from R45; value 51K -> 51k; footprint Resistor_SMD:R_0603_1608Metric -> P4Core:R_0603_1608Metric; moved to B.Cu
- R9: value 10R -> 10k; footprint Resistor_SMD:R_0603_1608Metric -> P4Local_Resistor_SMD:R_0603_1608Metric; moved to B.Cu
- SW1: value Card Detect -> EM-01KP; footprint Button_Switch_SMD:SW_DIP_SPSTx01_Slide_6.7x4.1mm_W8.61mm_P2.54mm_LowProfile -> P4Local_Button_Switch_SMD:SW_DIP_SPSTx01_Slide_6.7x4.1mm_W8.61mm_P2.54mm_LowProfile
- SW2: value RESET -> SKRPACE010; footprint SKRPACE010_C139797:SW_SKRPACE010_C139797 -> P4Local_SKRPACE010_C139797:SW_SKRPACE010_C139797
- SW3: value POWER -> SK-12D02-G030; footprint Button_Switch_THT:SW_Slide_SPDT_Angled_CK_OS102011MA1Q -> P4Local_Button_Switch_THT:SW_Slide_SPDT_Angled_CK_OS102011MA1Q
- TS1: value Touchscreen -> FH34SRJ-6S-0.5SH(50); footprint FT6236_TOUCH_6P:FT6236_TOUCH_6P_ALIGNED_V3 -> P4Local_FT6236_TOUCH:Hirose_FH34SRJ-6S-0.5SH_FT6236; moved to B.Cu
- U1: renamed from U4; footprint PCM_Espressif:ESP32-P4 -> P4Core:ESP32-P4; moved to B.Cu
- U2: value PCM5102 -> PCM5102APWR; footprint Package_SO:TSSOP-20_4.4x6.5mm_P0.65mm -> P4Local_Package_SO:TSSOP-20_4.4x6.5mm_P0.65mm; moved to B.Cu
- U3: footprint Package_DFN_QFN:QFN-28-1EP_4x4mm_P0.45mm_EP2.6x2.6mm -> P4Local_Package_DFN_QFN:QFN-28-1EP_4x4mm_P0.45mm_EP2.6x2.6mm; moved to B.Cu
- U5: value TLV62569DBV -> TLV62569DBVR; footprint Package_TO_SOT_SMD:SOT-23-5 -> P4Core:SOT-23-5; moved to B.Cu
- U6: footprint Package_SO:SOIC-8_5.3x5.3mm_P1.27mm -> P4Core:WSON-8-1EP_8x6mm_P1.27mm_EP3.4x4.3mm; moved to B.Cu
- U8: value TPS61183RTJT -> LD39150DT33-R; footprint Package_TO_SOT_SMD:SOT-23-5 -> P4Local_Package_TO_SOT_SMD:TO-252-3_TabPin2; moved to B.Cu
- U9: value ESP32-C6-MINI-1/U -> ESP32-C6-MINI-1-H4; footprint PCM_Espressif:ESP32-C6-MINI-1 -> P4Core:ESP32-C6-MINI-1; moved to B.Cu
- Y1: footprint Crystal:Crystal_SMD_3225-4Pin_3.2x2.5mm -> P4Core:Crystal_SMD_3225-4Pin_3.2x2.5mm; moved to B.Cu
- Y2: footprint Crystal:Crystal_SMD_3215-2Pin_3.2x1.5mm -> P4Core:Crystal_SMD_3215-2Pin_3.2x1.5mm; moved to B.Cu
- moved R9 521.5 mm to (145.0, 140.0)
- moved R50 514.8 mm to (137.0, 120.0), turned to -90 degrees
- moved R49 510.7 mm to (142.0, 120.5)
- moved R17 508.3 mm to (134.8, 108.0), turned to 90 degrees
- moved R59 506.1 mm to (142.5, 134.1), turned to 180 degrees
- moved R57 487.1 mm to (145.5, 135.0), turned to 180 degrees
- moved R58 478.4 mm to (142.5, 135.8), turned to 180 degrees
- moved R52 475.3 mm to (130.0, 103.0), turned to 90 degrees
- moved R5 470.3 mm to (129.5, 96.3), turned to 90 degrees
- moved R55 469.9 mm to (142.5, 137.4), turned to 180 degrees
- moved R56 469.2 mm to (145.5, 136.6), turned to 180 degrees
- moved R8 455.9 mm to (116.0, 132.3), turned to 180 degrees
- moved R54 454.1 mm to (145.5, 138.2), turned to 180 degrees
- moved R26 454.0 mm to (97.5, 104.0), turned to -90 degrees
- moved R46 436.6 mm to (70.5, 138.5), turned to 180 degrees
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Connections:
- net /GPIO54 renamed /C6_EN
- net /GPIO6 renamed /P4_C6_IO6
- C1 pad 1: /ES_CDATA -> /I2C_SDA
- C103 pad 1: /ESP_3V3 -> /LDO_3V3
- C104 pad 1: /ESP_3V3 -> /LDO_3V3
- C108 pad 1: /ESP_3V3 -> /LDO_3V3
- C109 pad 1: /ESP_3V3 -> /LDO_3V3
- C11 pad 1: Net-(U3-AVDD) -> /ES_AVDD
- C110 pad 1: /ESP_3V3 -> /LDO_3V3
- C111 pad 1: /ESP_3V3 -> /LDO_3V3
- C112 pad 1: /ESP_3V3 -> /LDO_3V3
- C114 pad 1: /ESP_3V3 -> /LDO_3V3
- C116 pad 1: /ESP_3V3 -> /ESP_LDO_VO1
- C117 pad 1: /ESP_3V3 -> /LDO_3V3
- C118 pad 1: /ESP_3V3 -> /LDO_3V3
- C119 pad 1: /ESP_3V3 -> /LDO_3V3
- C12 pad 1: Net-(U3-AVDD) -> /ES_AVDD
- C120 pad 1: /ESP_3V3 -> /LDO_3V3
- C123 pad 1: GND -> /XTAL_P
- C123 pad 2: /XTAL_P -> GND
- C124 pad 1: GND -> /XTAL_N
- C124 pad 2: /XTAL_N -> GND
- C125 pad 1: GND -> /P4_RTC0
- C125 pad 2: /GPIO0 -> GND
- C126 pad 1: GND -> /P4_RTC1
- C126 pad 2: /GPIO1 -> GND
- C127 pad 1: /ESP_3V3 -> GND
- C127 pad 2: GND -> /ESP_LDO_VO1
- C132 pad 1: /ESP_3V3 -> /LDO_3V3
- C133 pad 1: /ESP_3V3 -> /LDO_3V3
- C134 pad 1: /ESP_3V3 -> /LDO_3V3
- C19 pad 1: /REG_3V3 -> GND
- C19 pad 2: GND -> /LDO_3V3
- C2 pad 1: /ES_CCLK -> /I2C_SCL
- C20 pad 1: /REG_3V3 -> GND
- C20 pad 2: GND -> /LDO_3V3
- C21 pad 1: /REG_3V3 -> /LDO_3V3
- C22 pad 1: /REG_3V3 -> GND
- C22 pad 2: GND -> /VBAT
- C3 pad 1: /ES_MCLK -> Net-(C3-Pad1)
- C3 pad 2: GND -> /Headphone_L
- C4 pad 1: /ES_DVDD -> /ES8388_3V3
- C5 pad 1: /ES_DVDD -> /ES8388_3V3
- C6 pad 1: /ES_DVDD -> /ES8388_3V3
- C7 pad 1: /ES_LRCK -> Net-(C7-Pad1)
- C7 pad 2: GND -> /Headphone_R
- C95 pad 1: /ESP_3V3 -> /LDO_3V3
- C96 pad 1: /ESP_3V3 -> /LDO_3V3
- DS1 pad 12: unconnected-(DS1-RDX-Pad12) -> /LDO_3V3
- DS1 pad 38: /REG_3V3 -> /LDO_3V3
- DS1 pad 39: /REG_3V3 -> /LDO_3V3
- DS1 pad 40: /REG_3V3 -> /LDO_3V3
- DS1 pad 6: /REG_3V3 -> /LDO_3V3
- DS1 pad 7: /REG_3V3 -> /LDO_3V3
- J2 pad R2: unconnected-(J2-Ring_2-PadR2) -> GND
- J2 pad S: GND -> /HEADSET_MIC
- J5 pad 1: /USB_5V -> Net-(D3-K)
- J5 pad 2: /ESP_3V3 -> /USB_N
- J5 pad 3: /GPIO13 -> /USB_P
- J6 pad 4: Net-(J6-VDD) -> /SD_3V3
- J7 pad 1: /C6_IO9 -> /C6_BOOT
- J7 pad 2: GND -> /C6_RX
- J7 pad 3: /C6_U0RXD -> /C6_TX
- J7 pad 4: /C6_U0TXD -> GND
- L1 pad 1: /REG_3V3 -> /LDO_3V3
- L1 pad 2: /ES_DVDD -> /ES8388_3V3
- L2 pad 1: Net-(U5-SW) -> /ESP_VDD_HP
- L2 pad 2: /ESP_VDD_HP -> /P4_DCDC_SW
- Q2 pad 2: /ESP_3V3 -> /LDO_3V3
- Q2 pad 3: Net-(J6-VDD) -> /SD_3V3
- R1 pad 1: /REG_3V3 -> /LDO_3V3
- R1 pad 2: /ES_CCLK -> /I2C_SCL
- R17 pad 1: /FB_DCDC -> /I2S_MCLK
- R17 pad 2: GND -> /ES_MCLK
- R2 pad 1: /REG_3V3 -> /LDO_3V3
- R2 pad 2: /ES_CDATA -> /I2C_SDA
- R3 pad 1: /I2C_SCL -> /P4_STRAP36
- R3 pad 2: /ES_CCLK -> /LDO_3V3
- R36 pad 1: /ESP_3V3 -> /LDO_3V3
- R4 pad 1: /I2C_SDA -> /ES_AVDD
- R4 pad 2: /ES_CDATA -> /ES8388_3V3
- R46 pad 1: /ESP_3V3 -> /SD_3V3
- R5 pad 1: /I2S_MCLK -> /I2S_ASDOUT
- R5 pad 2: /ES_MCLK -> /ES_ASDOUT
- R51 pad 1: /GPIO0 -> /P4_RTC0
- R51 pad 2: /GPIO1 -> /P4_RTC1
- R52 pad 1: /FLASH_CS_A -> /ESP_LDO_VO1
- R52 pad 2: /ESP_3V3 -> /FLASH_CS_A
- R53 pad 1: /ESP_3V3 -> /LDO_3V3
- R54 pad 1: /GPIO17 -> /LDO_3V3
- R54 pad 2: /ESP_3V3 -> /P4_C6_IO17
- R55 pad 1: /GPIO16 -> /LDO_3V3
- R55 pad 2: /ESP_3V3 -> /P4_C6_IO16
- R56 pad 1: /GPIO15 -> /LDO_3V3
- R56 pad 2: /ESP_3V3 -> /P4_C6_IO15
- R57 pad 1: /GPIO18 -> /LDO_3V3
- R57 pad 2: /ESP_3V3 -> /P4_C6_IO18
- R58 pad 1: /GPIO14 -> /LDO_3V3
- R58 pad 2: /ESP_3V3 -> /P4_C6_IO14
- R59 pad 1: /GPIO19 -> /LDO_3V3
- R59 pad 2: /ESP_3V3 -> /P4_C6_IO19
- R9 pad 1: Net-(U3-AVDD) -> /C6_BOOT
- R9 pad 2: /REG_3V3 -> /LDO_3V3
- SW3 pad 3: /VBUS_5V -> /USB_PROTECTED_5V
- TS1 pad 1: /REG_3V3 -> /LDO_3V3
- U1 pad 1: /GPIO1 -> /P4_RTC1
- U1 pad 10: /I2S_MCLK -> /I2S_DSDIN
- U1 pad 101: /ESP_3V3 -> /LDO_3V3
- U1 pad 102: /ESP_3V3 -> /VBAT
- U1 pad 104: /GPIO0 -> /P4_RTC0
- U1 pad 11: /I2S_SCLK -> /I2S_LRCK
- U1 pad 12: /I2S_LRCK -> /I2S_ASDOUT
- U1 pad 13: /I2S_DSDIN -> /I2S_BCLK
- U1 pad 15: /GPIO14 -> /P4_C6_IO14
- U1 pad 16: /GPIO15 -> /P4_C6_IO15
- U1 pad 17: /GPIO16 -> /P4_C6_IO16
- U1 pad 18: /GPIO17 -> /P4_C6_IO17
- U1 pad 19: /GPIO18 -> /P4_C6_IO18
- U1 pad 20: /GPIO19 -> /P4_C6_IO19
- U1 pad 21: /ESP_3V3 -> /LDO_3V3
- U1 pad 22: /GPIO20 -> /PCM_DATA
- U1 pad 23: /GPIO21 -> /PCM_BCLK
- U1 pad 25: /GPIO23 -> /PCM_LRCK
- U1 pad 3: /PCM_BCK -> /GPIO3
- U1 pad 30: /ESP_3V3 -> /ESP_LDO_VO1
- U1 pad 4: /PCM_DATA -> /GPIO4
- U1 pad 5: /PCM_LRCK -> /GPIO5
- U1 pad 51: /ESP_3V3 -> /LDO_3V3
- U1 pad 57: /GPIO28 -> /TFT_MISO
- U1 pad 58: /GPIO29 -> /TFT_SCK
- U1 pad 60: /GPIO30 -> /TFT_MOSI
- U1 pad 61: /GPIO31 -> /TFT_DC
- U1 pad 62: /ESP_3V3 -> /LDO_3V3
- U1 pad 63: /GPIO32 -> /I2S_MCLK
- U1 pad 64: /GPIO33 -> /TCH_RST
- U1 pad 66: GND -> /ESP_BOOT
- U1 pad 68: Net-(U4-GPIO36) -> /P4_STRAP36
- U1 pad 69: /GPIO37 -> /U0RXD
- U1 pad 70: /GPIO38 -> /U0TXD
- U1 pad 75: /ESP_3V3 -> /LDO_3V3
- U1 pad 77: /ESP_3V3 -> /LDO_3V3
- U1 pad 87: /TCH_INT -> unconnected-(U1-GPIO45-Pad87)
- U1 pad 88: /TCH_RST -> unconnected-(U1-GPIO46-Pad88)
- U1 pad 89: /TFT_MISO -> /TCH_INT
- U1 pad 9: /ESP_3V3 -> /LDO_3V3
- U1 pad 90: /TFT_SCK -> unconnected-(U1-GPIO48-Pad90)
- U1 pad 92: /TFT_MOSI -> /GPIO49
- U1 pad 93: /TFT_RESET -> /GPIO50
- U1 pad 94: /TFT_DC -> /TFT_RESET
- U1 pad 96: /ESP_3V3 -> /LDO_3V3
- U2 pad 1: /REG_3V3 -> /LDO_3V3
- U2 pad 13: /PCM_BCK -> /PCM_BCLK
- U2 pad 20: /REG_3V3 -> /LDO_3V3
- U2 pad 8: /REG_3V3 -> /LDO_3V3
- U3 pad 16: /REG_3V3 -> /ES8388_3V3
- U3 pad 17: Net-(U3-AVDD) -> /ES_AVDD
- U3 pad 2: /ES_DVDD -> /ES8388_3V3
- U3 pad 23: unconnected-(U3-RIN1-Pad23) -> /ADC_MIC_N
- U3 pad 24: unconnected-(U3-LIN1-Pad24) -> /ADC_MIC_P
- U3 pad 26: /REG_3V3 -> /LDO_3V3
- U3 pad 27: /ES_CDATA -> /I2C_SDA
- U3 pad 28: /ES_CCLK -> /I2C_SCL
- U3 pad 3: /ES_DVDD -> /ES8388_3V3
- U3 pad 5: /ES_SCLK -> /ES_BCLK
- U3 pad 8: unconnected-(U3-ASDOUT-Pad8) -> /ES_ASDOUT
- U5 pad 3: Net-(U5-SW) -> /P4_DCDC_SW
- U5 pad 4: /ESP_3V3 -> /LDO_3V3
- U6 pad 8: /ESP_3V3 -> /ESP_LDO_VO1
- U8 pad 3: /USB_5V -> /LDO_3V3
- U9 pad 22: Net-(U9-GPIO8) -> /C6_STRAP8
- U9 pad 23: /C6_IO9 -> /C6_BOOT
- U9 pad 24: /GPIO19 -> /P4_C6_IO19
- U9 pad 25: /GPIO18 -> /P4_C6_IO18
- U9 pad 26: /GPIO14 -> /P4_C6_IO14
- U9 pad 27: /GPIO15 -> /P4_C6_IO15
- U9 pad 28: /GPIO16 -> /P4_C6_IO16
- U9 pad 29: /GPIO17 -> /P4_C6_IO17
- U9 pad 3: /ESP_3V3 -> /LDO_3V3
- U9 pad 30: /C6_U0RXD -> /C6_RX
- U9 pad 31: /C6_U0TXD -> /C6_TX
- Y1 pad 1: /XTAL_P -> /XTAL_N
- Y1 pad 3: /XTAL_N -> /XTAL_P
- Y2 pad 1: /GPIO1 -> /P4_RTC0
- Y2 pad 2: /GPIO0 -> /P4_RTC1
Routing:
- net GND: track 0.00 -> 209.5 mm, vias 0 -> 188
- net /VBAT: track 0.00 -> 177.0 mm, vias 0 -> 6
- net /ESP_EN: track 0.00 -> 155.1 mm, vias 0 -> 10
- net /I2C_SDA: track 0.00 -> 153.5 mm, vias 0 -> 13
- net /I2C_SCL: track 0.00 -> 138.6 mm, vias 0 -> 12
- net /ESP_BOOT: track 0.00 -> 132.1 mm, vias 0 -> 7
- net /SD1_D3: track 0.00 -> 128.9 mm, vias 0 -> 11
- net /SD1_CMD: track 0.00 -> 128.0 mm, vias 0 -> 9
- net /U0TXD: track 0.00 -> 127.6 mm, vias 0 -> 12
- net /U0RXD: track 0.00 -> 124.5 mm, vias 0 -> 6
- net /SD1_CLK: track 0.00 -> 124.1 mm, vias 0 -> 10
- net /SD1_D0: track 0.00 -> 124.1 mm, vias 0 -> 10
- net /SD1_D2: track 0.00 -> 121.2 mm, vias 0 -> 13
- net /SD1_D1: track 0.00 -> 118.1 mm, vias 0 -> 15
- net /C6_RX: track 0.00 -> 116.3 mm, vias 0 -> 3
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- added copper zone on In1.Cu, net /ESP_VDD_HP
- added copper zone on B.Cu, net /LDO_3V3
- added copper zone on In1.Cu, net /LDO_3V3
- added copper zone on B.Cu, net /SD_3V3
- added copper zone on In1.Cu, net /SD_3V3
- added copper zone on In1.Cu, net /USB_5V
- added copper zone on In1.Cu, net /USB_PROTECTED_5V
- added copper zone on In1.Cu, net /VBUS_5V
- added copper zone on B.Cu, net GND
- added copper zone on F.Cu, net GND
- added copper zone on In2.Cu, net GND
Other:
- board size 108 x 60.9 mm -> 100 x 85.4 mm
- board text added: "3.3V"
- board text added: "3V3"
- board text added: "5V"
- board text added: "BOOT"
- board text added: "CELL"
- board text added: "CONTROL"
- board text added: "ESP_BOOT"
- board text added: "ESP_EN"
- board text added: "GND"
- board text added: "GPIO"
- board text added: "GPIO13"
- board text added: "GPIO2(SCK)"
- board text added: "GPIO22"
- board text added: "GPIO3(MOSI)"
- board text added: "GPIO34"
- board text added: "GPIO4(MISO)"
- board text added: "GPIO49"
- board text added: "GPIO5(CS)"
- board text added: "GPIO50"
- board text added: "GPIO7(SDA)"
- board text added: "GPIO8(SCL)"
- board text added: "I2C"
- board text added: "P4-WSM32-AT4SC6 V1.0"
- board text added: "RESET"
- board text added: "RTC"
- board text added: "RX"
- board text added: "SPI"
- board text added: "TX"
- board text added: "U0RXD"
- board text added: "U0TXD"
- board text added: "UART"
- board text added: "VBAT"
