File: KiCAD PCB Files/P4-Audio-TFT/P4-Audio-TFT.kicad_sch (KiCad schematic)
At the start: 113 parts, among them J1 USB-C Program, J2 Headphone, J3 Type A Host, J4 Line-Out, SW1 RESET, SW3 BOOT, U2 PCM5102, U3 ES8388, U5 TLV62569DBV, U6 W25Q256JV, U7 TLV62569DBV, U8 TPS7A20xxxDBV, Y1 40Mhz, Y2 32.768Khz

Commit message: PCB Design started
Parts:
- removed C17, C18: 100uF, symbol Device:C
- removed C65, C66: 0.1uF, PCM_Espressif:ESP32-P4, symbol Device:C
- removed J2: Headphone, symbol Connector_Audio:AudioJack3
- removed J4: Line-Out, symbol Connector_Audio:AudioJack3
- removed SW1: RESET, Button_Switch_THT:SW_NKK_GW12LJP, symbol Switch:SW_Push
- removed SW3: BOOT, Button_Switch_THT:SW_NKK_GW12LJP, symbol Switch:SW_Push
- removed Y1: 40Mhz, Package_DIP:DIP-40_W15.24mm, symbol Device:Crystal
- added C69, C70, C73, C74, C77, C78: 0.1uF, Capacitor_SMD:C_0603_1608Metric, symbol Device:C
- added C71, C76, C79: 10uF, Capacitor_SMD:C_0603_1608Metric, symbol Device:C
- added C72: 22uF, Capacitor_SMD:C_0603_1608Metric, symbol Device:C
- added C75, C80: 1uF, Capacitor_SMD:C_0603_1608Metric, symbol Device:C
- added C83, C84: 100uF, Capacitor_SMD:CP_Elec_6.3x5.8, symbol Device:C_Polarized
- added D1: LED, LED_SMD:LED_0603_1608Metric, symbol Device:LED
- added D3: SS36, Diode_SMD:D_SMA, symbol Device:D
- added DS1: ILI TFT Panel, ILI9488_TFT_40P:ILI9488_TFT_40P_ALIGNED_V3, symbol ILI9488_4IN_TFT_40P:ILI9488_4IN_TFT_40P
- added H1, H2, H3, H4: (no value), MountingHole:MountingHole_3.2mm_M3, symbol Mechanical:MountingHole
- added J2: Headphone, Connector_Audio:Jack_3.5mm_PJ320D_Horizontal, symbol PJ320D_KiCad10:AudioJack_PJ320D
- added J4: Line-Out, Connector_Audio:Jack_3.5mm_PJ320D_Horizontal, symbol PJ320D_KiCad10:AudioJack_PJ320D
- added J5: EXPANSION, Connector_PinSocket_2.54mm:PinSocket_2x10_P2.54mm_Vertical, symbol Connector_Generic:Conn_02x10_Odd_Even
- added J6: Micro_SD_Card, Connector_Card:microSD_HC_Hirose_DM3AT-SF-PEJM5, symbol Connector:Micro_SD_Card
- added J7: C6 PROG, Connector_PinHeader_2.54mm:PinHeader_1x04_P2.54mm_Vertical, symbol Connector:Conn_01x04_Pin
- added Q1: EMH4T2R, Package_TO_SOT_SMD:SOT-563, symbol EMH4T2R:EMH4T2R
- added Q2: AO3401A, Package_TO_SOT_SMD:SOT-23, symbol Transistor_FET:Q_PMOS_GSD
- added Q3: AO3400A, Package_TO_SOT_SMD:SOT-23, symbol Transistor_FET:Q_NMOS_GSD
- added R28, R29, R30, R31, R32, R33, R34, R35, R36, R37, R38, R39, R46: 10K, Resistor_SMD:R_0603_1608Metric, symbol Device:R
- added R40, R41, R42, R43, R44, R45: 51K, Resistor_SMD:R_0603_1608Metric, symbol Device:R
- added SW1: Card Detect, Button_Switch_SMD:SW_DIP_SPSTx01_Slide_6.7x4.1mm_W8.61mm_P2.54mm_LowProfile, symbol Switch:SW_DIP_x01
- added SW2: RESET, SKRPACE010_C139797:SW_SKRPACE010_C139797, symbol Switch:SW_Push
- added SW3: POWER, Button_Switch_THT:SW_Slide_SPDT_Angled_CK_OS102011MA1Q, symbol Switch:SW_SPDT
- added TS1: Touchscreen, FT6236_TOUCH_6P:FT6236_TOUCH_6P_ALIGNED_V3, symbol FT6236_TOUCH_6P:FT6236_TOUCH_6P
- added U1: CH340C, Package_SO:SOIC-16_3.9x9.9mm_P1.27mm, symbol Interface_USB:CH340C
- added U9: ESP32-C6-MINI-1/U, PCM_Espressif:ESP32-C6-MINI-1, symbol PCM_Espressif:ESP32-C6-MINI-1/U
- added Y1: 40Mhz, Crystal:Crystal_SMD_3225-4Pin_3.2x2.5mm, symbol Crystal_4Pin_GND24_KiCad10:Crystal_4Pin_GND24
- C1, C2: footprint (none) -> Capacitor_SMD:C_0603_1608Metric; KiLib_Generator (none) -> SMD_2terminal_chip_molded; LCSC (none) -> C376776
- C10, C12, C4: footprint (none) -> Capacitor_SMD:C_0603_1608Metric; KiLib_Generator (none) -> SMD_2terminal_chip_molded; LCSC (none) -> C277476
- C11, C5, C6, C9: footprint (none) -> Capacitor_SMD:C_0603_1608Metric; KiLib_Generator (none) -> SMD_2terminal_chip_molded; LCSC (none) -> C14663
- C13, C15, C19, C20, C21, C25: value 100nF -> 0.1uF; footprint (none) -> Capacitor_SMD:C_0603_1608Metric; KiLib_Generator (none) -> SMD_2terminal_chip_molded; LCSC (none) -> C14663
- C14, C16, C22: footprint (none) -> Capacitor_SMD:C_0603_1608Metric; KiLib_Generator (none) -> SMD_2terminal_chip_molded; LCSC (none) -> C96446
- C23, C29, C30, C38, C39, C41, C43, C44, C46, C48, C49, C51, C52, C61, C68: footprint PCM_Espressif:ESP32-P4 -> Capacitor_SMD:C_0603_1608Metric; KiLib_Generator (none) -> SMD_2terminal_chip_molded; LCSC (none) -> C14663
- C24, C26: footprint (none) -> Capacitor_SMD:C_0603_1608Metric; KiLib_Generator (none) -> SMD_2terminal_chip_molded; LCSC (none) -> C99228
- C27, C28: footprint (none) -> Capacitor_SMD:C_0603_1608Metric; KiLib_Generator (none) -> SMD_2terminal_chip_molded; LCSC (none) -> C54421959
- C3, C7, C8: footprint (none) -> Capacitor_SMD:C_0603_1608Metric; KiLib_Generator (none) -> SMD_2terminal_chip_molded; LCSC (none) -> C1658
- C31, C32, C33, C34, C36, C50: footprint PCM_Espressif:ESP32-P4 -> Capacitor_SMD:C_0603_1608Metric; KiLib_Generator (none) -> SMD_2terminal_chip_molded; LCSC (none) -> C106248
- C35, C37: value 0.1UF -> 0.1uF; footprint PCM_Espressif:ESP32-P4 -> Capacitor_SMD:C_0603_1608Metric; KiLib_Generator (none) -> SMD_2terminal_chip_molded; LCSC (none) -> C14663
- C40, C42, C45, C47, C62, C64, C67: footprint PCM_Espressif:ESP32-P4 -> Capacitor_SMD:C_0603_1608Metric; KiLib_Generator (none) -> SMD_2terminal_chip_molded; LCSC (none) -> C96446
- C53, C54: footprint PCM_Espressif:ESP32-P4 -> Capacitor_SMD:C_0603_1608Metric; KiLib_Generator (none) -> SMD_2terminal_chip_molded; LCSC (none) -> C277476
- C55: footprint PCM_Espressif:ESP32-P4 -> Capacitor_SMD:C_0603_1608Metric; KiLib_Generator (none) -> SMD_2terminal_chip_molded; LCSC (none) -> C2762594
- C56, C57, C58, C59, C60: footprint PCM_Espressif:ESP32-P4 -> Capacitor_SMD:C_0603_1608Metric; KiLib_Generator (none) -> SMD_2terminal_chip_molded; LCSC (none) -> C376775
- C63: value 22pF -> 6.8pF; footprint PCM_Espressif:ESP32-P4 -> Capacitor_SMD:C_0603_1608Metric; KiLib_Generator (none) -> SMD_2terminal_chip_molded; LCSC (none) -> C1679
- J1: footprint (none) -> Connector_USB:USB_C_Receptacle_HRO_TYPE-C-31-M-12; LCSC (none) -> C165948
- J3: value Type A Host -> Type B Host; footprint Package_TO_SOT_SMD:SOT-23-5 -> Connector_USB:USB_A_Molex_67643_Horizontal; LCSC (none) -> C2765194
- L1: footprint (none) -> Inductor_SMD:L_0603_1608Metric; KiLib_Generator (none) -> SMD_2terminal_chip_molded; LCSC (none) -> C107335
- L2: value 2.2uH -> 1uH 2.5*2*1.2 3.5A; footprint Package_TO_SOT_SMD:SOT-23-5 -> Inductor_SMD:L_0805_2012Metric; KiLib_Generator (none) -> SMD_2terminal_chip_molded; LCSC (none) -> C53514708
- L3: footprint Package_TO_SOT_SMD:SOT-23-5 -> Inductor_SMD:L_0805_2012Metric; KiLib_Generator (none) -> SMD_2terminal_chip_molded; LCSC (none) -> C42455275
- R1, R2: footprint (none) -> Resistor_SMD:R_0603_1608Metric; KiLib_Generator (none) -> SMD_2terminal_chip_molded; LCSC (none) -> C21190
- R10, R11: footprint (none) -> Resistor_SMD:R_0603_1608Metric; KiLib_Generator (none) -> SMD_2terminal_chip_molded; LCSC (none) -> C23345
- R12, R25: footprint (none) -> Resistor_SMD:R_0603_1608Metric; KiLib_Generator (none) -> SMD_2terminal_chip_molded; LCSC (none) -> C25804
- R13, R14: footprint (none) -> Resistor_SMD:R_0603_1608Metric; KiLib_Generator (none) -> SMD_2terminal_chip_molded; LCSC (none) -> C23179
- R15: value 33 -> 100R; footprint (none) -> Resistor_SMD:R_0603_1608Metric; LCSC (none) -> C105588
- R16: value 10K -> 5.1K; footprint (none) -> Resistor_SMD:R_0603_1608Metric; KiLib_Generator (none) -> SMD_2terminal_chip_molded; LCSC (none) -> C23186
- R17, R22: value 499K -> 200K; footprint (none) -> Resistor_SMD:R_0603_1608Metric; KiLib_Generator (none) -> SMD_2terminal_chip_molded; LCSC (none) -> C25811
- R18: footprint (none) -> Resistor_SMD:R_0603_1608Metric; KiLib_Generator (none) -> SMD_2terminal_chip_molded; LCSC (none) -> C7250
- R19: footprint Package_QFP:LQFP-100_14x14mm_P0.5mm -> Resistor_SMD:R_0603_1608Metric; KiLib_Generator (none) -> SMD_2terminal_chip_molded; LCSC (none) -> C25804
- R20: footprint (none) -> Resistor_SMD:R_0603_1608Metric; KiLib_Generator (none) -> SMD_2terminal_chip_molded; LCSC (none) -> C25803
- R21: value 22.1K -> 22K1; footprint (none) -> Resistor_SMD:R_0603_1608Metric; KiLib_Generator (none) -> SMD_2terminal_chip_molded; LCSC (none) -> C227715
- R23: value 10K -> 100K; footprint Package_QFP:LQFP-100_14x14mm_P0.5mm -> Resistor_SMD:R_0603_1608Metric; LCSC (none) -> C25803
- R24, R27: footprint (none) -> Resistor_SMD:R_0603_1608Metric; KiLib_Generator (none) -> SMD_2terminal_chip_molded; LCSC (none) -> C23186
- R26: value 10K -> 16R; footprint (none) -> Resistor_SMD:R_1206_3216Metric; LCSC (none) -> C2974063
- R3, R4: footprint (none) -> Resistor_SMD:R_0603_1608Metric; KiLib_Generator (none) -> SMD_2terminal_chip_molded; LCSC (none) -> C23138
- R5, R6, R7, R8: footprint (none) -> Resistor_SMD:R_0603_1608Metric; KiLib_Generator (none) -> SMD_2terminal_chip_molded; LCSC (none) -> C23140
- R9: footprint (none) -> Resistor_SMD:R_0603_1608Metric; KiLib_Generator (none) -> SMD_2terminal_chip_molded; LCSC (none) -> C22859
- U2: KiLib_Generator (none) -> package/gullwing; LCSC (none) -> C107671
- U3: KiLib_Generator (none) -> package/no_lead; LCSC (none) -> C365736
- U4: value (none) -> ESP32-P4NRW32X; LCSC (none) -> C54540373
- U5, U7: KiLib_Generator (none) -> package/gullwing; LCSC (none) -> C141836
- U6: value W25Q256JV -> W25Q256JVEIQ; KiLib_Generator (none) -> package/no_lead; LCSC (none) -> C97522
- U8: value TPS7A20xxxDBV -> TPS61183RTJT; LCSC (none) -> C2862740
- Y2: footprint Package_DIP:DIP-40_W15.24mm -> Crystal:Crystal_SMD_3215-2Pin_3.2x1.5mm; LCSC (none) -> C32346
Connections:
- net GPIO26 is gone; now on net USB_N: U4.55 (GPIO26/USB1P1_N1)
- net GPIO27 is gone; now on net USB_P: U4.56 (GPIO27/USB1P1_P1)
- net GPIO_0 is gone; now on net GPIO0: U4.104 (GPIO0)
- net ESP_3V3: now also C50.1, C51.1, C61.1, R19.2, R25.1, U4.30 (VDD_FLASH_IO), U6.8 (VCC), C70.1, C71.1, C74.1, C78.1, C79.1, J5.2 (Pin_2), Q2.2 (S), R28.1, R29.1, R30.1, R31.1, R32.1, R33.1, R34.1, R35.1, R36.1, R38.1, R39.2, R40.2, R41.2, R42.2, R43.2, R44.2, R45.2, R46.1, U1.16 (VCC), U1.4 (V3), U9.3 (3V3); no longer R23.2, R25.2, R26.2
- net ESP_EN: now also C75.1, J5.17 (Pin_17), Q1.6 (C1), R29.2, SW2.1; no longer R23.1
- net ESP_LDO_VO1: no longer C50.1, C51.1, C61.1, R19.2, U4.30 (VDD_FLASH_IO), U6.8 (VCC)
- net ESP_VDD_HP: now also C72.1, C73.1
- net GND: now also R23.1, R25.2, U4.66 (GPIO35), C69.2, C70.2, C71.2, C72.2, C73.2, C74.2, C75.2, C76.2, C77.2, C78.2, C79.2, C80.2, D1.1 (K), DS1.16 (GND), DS1.37 (GND), DS1.5 (GND), J2.S (Sleeve), J4.S (Sleeve), J5.16 (Pin_16), J5.18 (Pin_18), J5.19 (Pin_19), J5.20 (Pin_20), J5.4 (Pin_4), J5.5 (Pin_5), J6.6 (VSS), J6.9 (CD_A), J6.SH (SHIELD), J7.2 (Pin_2), Q1.3 (C2), Q3.2 (S), R37.1, SW2.2, TS1.6 (GND), U1.1 (GND), U9.1 (GND), U9.11 (GND), U9.14 (GND), U9.2 (GND), U9.36 (GND), U9.37 (GND), U9.38 (GND), U9.39 (GND), U9.40 (GND), U9.41 (GND), U9.42 (GND), U9.43 (GND), U9.44 (GND), U9.45 (GND), U9.46 (GND), U9.47 (GND), U9.48 (GND), U9.49 (GND), U9.50 (GND), U9.51 (GND), U9.52 (GND), U9.53 (GND), Y1.2 (GND), Y1.4 (GND)
- net GPIO13: now also J5.3 (Pin_3), SW1.1
- net GPIO14: now also R44.1, U9.26 (GPIO20)
- net GPIO15: now also R42.1, U9.27 (GPIO21)
- net GPIO16: now also R41.1, U9.28 (GPIO22)
- net GPIO17: now also R40.1, U9.29 (GPIO23)
- net GPIO18: now also R43.1, U9.25 (GPIO19)
- net GPIO19: now also R45.1, U9.24 (GPIO18)
- net GPIO2: now also R15.1
- net GPIO20: now also J5.6 (Pin_6)
- net GPIO21: now also J5.7 (Pin_7)
- net GPIO22: now also J5.8 (Pin_8)
- net GPIO23: now also J5.9 (Pin_9)
- net GPIO28: now also J5.10 (Pin_10)
- net GPIO29: now also J5.11 (Pin_11)
- net GPIO30: now also J5.12 (Pin_12)
- net GPIO31: now also J5.13 (Pin_13)
- net GPIO32: now also J5.14 (Pin_14)
- net GPIO33: now also J5.15 (Pin_15)
- net GPIO53: now also Q2.1 (G), R36.2, R37.2
- net GPIO54: now also C80.1, R38.2, U9.8 (EN/CHIP_PU)
- net GPIO6: now also U9.5 (GPIO2/ADC1_CH2)
- net Headphone_L: now also C83.2, J2.T (Tip)
- net Headphone_R: now also C84.2, J2.R1 (Ring_1)
- net I2C_SCL: now also TS1.3 (SCL)
- net I2C_SDA: now also TS1.2 (SDA)
- net Lineout_L: now also J4.T (Tip)
- net Lineout_R: now also J4.R1 (Ring_1)
- net REG_3V3: now also DS1.38 (IM0), DS1.39 (IM1), DS1.40 (IM2), DS1.6 (VDDI), DS1.7 (VDD), TS1.1 (VDD)
- net SD1_CLK: now also J6.5 (CLK), R33.2
- net SD1_CMD: now also J6.3 (CMD), R32.2
- net SD1_D0: now also J6.7 (DAT0), R34.2
- net SD1_D1: now also J6.8 (DAT1), R46.2
- net SD1_D2: now also J6.1 (DAT2), R30.2
- net SD1_D3: now also J6.2 (DAT3/CD), R31.2
- net USB_5V: now also R26.1, U7.1 (EN), C69.1, D3.2 (A), J5.1 (Pin_1), SW3.2 (B); no longer J1.A4 (VBUS), J1.A9 (VBUS), J1.B4 (VBUS), J1.B9 (VBUS), J3.1 (VBUS)
- net USB_N: now also J3.2 (D-); no longer J1.A7 (D-), J1.B7 (D-), R15.2
- net USB_P: now also J3.3 (D+); no longer J1.A6 (D+), J1.B6 (D+), U4.53 (GPIO25/USB1P1_P0)
- net XTAL_N: now also Y1.3 (XTAL2)
- net XTAL_P: now also Y1.1 (XTAL1)
- net at R11.2: now also C84.1
- net at R16.2: now also D1.2 (A); no longer U7.1 (EN)
- net at R10.2: now also C83.1
- net at U4.52 (GPIO24/USB1P1_N0): no longer R15.1
- net GPIO34_BOOTMODE renamed GPIO34
- removed net GPIO35_BOOTMODE: R26.1, U4.66 (GPIO35)
- net GPIO36_BOOTMODE: no longer names the net of U4.68 (GPIO36)
- net GPIO36_BOOTMODE: now also R28.2; no longer R25.1
- net GPIO37_BOOTMODE renamed GPIO37
- net GPIO37: now also U1.3 (RXD)
- net GPIO38_BOOTMODE renamed GPIO38
- net GPIO38: now also U1.2 (TXD)
- net GPIO45 renamed TCH_INT
- net TCH_INT: now also TS1.4 (INT)
- net GPIO46 renamed TCH_RST
- net TCH_RST: now also TS1.5 (RST)
- net GPIO47 renamed TFT_MISO
- net TFT_MISO: now also DS1.14 (SPI_MISO)
- net GPIO48 renamed TFT_SCK
- net TFT_SCK: now also DS1.11 (WRX_SPI_SCLK)
- net GPIO49 renamed TFT_MOSI
- net TFT_MOSI: now also DS1.13 (SPI_MOSI)
- net GPIO50 renamed TFT_RESET
- net TFT_RESET: now also DS1.15 (RESET)
- net GPIO51 renamed TFT_DC
- net TFT_DC: now also DS1.10 (DCX_SPI_DC)
- net GPIO52 renamed TFT_CS
- net TFT_CS: now also DS1.9 (CSX_SPI_CS)
- net USBH_DM: no longer names the net of U4.49 (USB-DM)
- net USBH_DM: no longer J3.2 (D-)
- net USBH_DP: no longer names the net of U4.50 (USB-DP)
- net USBH_DP: no longer J3.3 (D+)
- new net: J6.10 (CD_B), R35.2, SW1.2
- new net: C76.1, C77.1, J6.4 (VDD), Q2.3 (D)
- new net: DS1.33 (LED_A), R26.2
- new net: Q3.1 (G), R15.2, R23.2
- new net: R39.1, U9.22 (GPIO8)
- new net: D3.1 (K), J3.1 (VBUS)
- new net C6_IO9: J7.1 (Pin_1), U9.23 (GPIO9)
- new net C6_U0RXD: J7.3 (Pin_3), U9.30 (U0RXD/GPIO17)
- new net C6_U0TXD: J7.4 (Pin_4), U9.31 (U0TXD/GPIO16)
- new net DTR: Q1.2 (IN1), Q1.4 (E2), U1.13 (~{DTR})
- new net LED_K: DS1.34 (LED_K), DS1.35 (LED_K), DS1.36 (LED_K), Q3.3 (D)
- new net RTS: Q1.1 (E1), Q1.5 (IN2), U1.14 (~{RTS})
- new net USBC_N: J1.A7 (D-), J1.B7 (D-), U1.6 (UD-)
- new net USBC_P: J1.A6 (D+), J1.B6 (D+), U1.5 (UD+)
- new net VBUS_5V: J1.A4 (VBUS), J1.A9 (VBUS), J1.B4 (VBUS), J1.B9 (VBUS), SW3.3 (C)
- no-connect marks 24 -> 64
Other:
- moved on the sheet: C10, C11, C12, C13, C14, C15, C16, C19, C20, C21, C22, C23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

Commit message: PCB WS and P4-C6 complete
Parts:
- removed C1, C2: 220pF, Capacitor_SMD:C_0603_1608Metric, symbol Device:C
- removed C10, C12, C4, C53, C54: 4.7uF, Capacitor_SMD:C_0603_1608Metric, symbol Device:C
- removed C11, C13, C15, C19, C20, C21, C23, C25, C29, C30, C35, C37, C38, C39, C41, C43, C44, C46, C48, C49, C5, C51, C52, C6, C61, C68, C69, C70, C73, C74, C77, C78, C9: 0.1uF, Capacitor_SMD:C_0603_1608Metric, symbol Device:C
- removed C14, C16, C22, C40, C42, C45, C47, C62, C64, C67, C71, C76, C79: 10uF, Capacitor_SMD:C_0603_1608Metric, symbol Device:C
- removed C24, C26: 2.2uF, Capacitor_SMD:C_0603_1608Metric, symbol Device:C
- removed C27, C28: 2.2nF, Capacitor_SMD:C_0603_1608Metric, symbol Device:C
- removed C3: 30pF, Capacitor_SMD:C_0603_1608Metric, symbol Device:C
- removed C31, C32, C33, C34, C36, C50, C75, C80: 1uF, Capacitor_SMD:C_0603_1608Metric, symbol Device:C
- removed C55, C72: 22uF, Capacitor_SMD:C_0603_1608Metric, symbol Device:C
- removed C56, C57, C58, C59, C60: 22pF, Capacitor_SMD:C_0603_1608Metric, symbol Device:C
- removed C63: 6.8pF, Capacitor_SMD:C_0603_1608Metric, symbol Device:C
- removed C7, C8: 30PF, Capacitor_SMD:C_0603_1608Metric, symbol Device:C
- removed C83, C84: 100uF, Capacitor_SMD:CP_Elec_6.3x5.8, symbol Device:C_Polarized
- removed D1: LED, LED_SMD:LED_0603_1608Metric, symbol Device:LED
- removed D3: SS36, Diode_SMD:D_SMA, symbol Device:D
- removed DS1: ILI TFT Panel, ILI9488_TFT_40P:ILI9488_TFT_40P_ALIGNED_V3, symbol ILI9488_4IN_TFT_40P:ILI9488_4IN_TFT_40P
- removed H1, H2, H3, H4: (no value), MountingHole:MountingHole_3.2mm_M3, symbol Mechanical:MountingHole
- removed J1: USB-C Program, Connector_USB:USB_C_Receptacle_HRO_TYPE-C-31-M-12, symbol Connector:USB_C_Receptacle_USB2.0_16P
- removed J2: Headphone, Connector_Audio:Jack_3.5mm_PJ320D_Horizontal, symbol PJ320D_KiCad10:AudioJack_PJ320D
- removed J3: Type B Host, Connector_USB:USB_A_Molex_67643_Horizontal, symbol Connector:USB_A
- removed J4: Line-Out, Connector_Audio:Jack_3.5mm_PJ320D_Horizontal, symbol PJ320D_KiCad10:AudioJack_PJ320D
- removed J5: EXPANSION, Connector_PinSocket_2.54mm:PinSocket_2x10_P2.54mm_Vertical, symbol Connector_Generic:Conn_02x10_Odd_Even
- removed J6: Micro_SD_Card, Connector_Card:microSD_HC_Hirose_DM3AT-SF-PEJM5, symbol Connector:Micro_SD_Card
- removed J7: C6 PROG, Connector_PinHeader_2.54mm:PinHeader_1x04_P2.54mm_Vertical, symbol Connector:Conn_01x04_Pin
- removed L1: 600R@100Mhz, Inductor_SMD:L_0603_1608Metric, symbol Device:L_Ferrite
- removed L2: 1uH 2.5*2*1.2 3.5A, Inductor_SMD:L_0805_2012Metric, symbol Device:L
- removed L3: 2.2uH, Inductor_SMD:L_0805_2012Metric, symbol Device:L
- removed Q1: EMH4T2R, Package_TO_SOT_SMD:SOT-563, symbol EMH4T2R:EMH4T2R
- removed Q2: AO3401A, Package_TO_SOT_SMD:SOT-23, symbol Transistor_FET:Q_PMOS_GSD
- removed Q3: AO3400A, Package_TO_SOT_SMD:SOT-23, symbol Transistor_FET:Q_NMOS_GSD
- removed R1, R2: 1K, Resistor_SMD:R_0603_1608Metric, symbol Device:R
- removed R10, R11: 22R, Resistor_SMD:R_0603_1608Metric, symbol Device:R
- removed R12, R19, R25, R28, R29, R30, R31, R32, R33, R34, R35, R36, R37, R38, R39, R46: 10K, Resistor_SMD:R_0603_1608Metric, symbol Device:R
- removed R13, R14: 470R, Resistor_SMD:R_0603_1608Metric, symbol Device:R
- removed R15: 100R, Resistor_SMD:R_0603_1608Metric, symbol Device:R
- removed R16, R24, R27: 5.1K, Resistor_SMD:R_0603_1608Metric, symbol Device:R
- removed R17, R22: 200K, Resistor_SMD:R_0603_1608Metric, symbol Device:R
- removed R18: 10M, Resistor_SMD:R_0603_1608Metric, symbol Device:R
- removed R20, R23: 100K, Resistor_SMD:R_0603_1608Metric, symbol Device:R
- removed R21: 22K1, Resistor_SMD:R_0603_1608Metric, symbol Device:R
- removed R26: 16R, Resistor_SMD:R_1206_3216Metric, symbol Device:R
- removed R3, R4: 330, Resistor_SMD:R_0603_1608Metric, symbol Device:R
- removed R40, R41, R42, R43, R44, R45: 51K, Resistor_SMD:R_0603_1608Metric, symbol Device:R
- removed R5, R6, R7, R8: 33R, Resistor_SMD:R_0603_1608Metric, symbol Device:R
- removed R9: 10R, Resistor_SMD:R_0603_1608Metric, symbol Device:R
- removed SW1: Card Detect, Button_Switch_SMD:SW_DIP_SPSTx01_Slide_6.7x4.1mm_W8.61mm_P2.54mm_LowProfile, symbol Switch:SW_DIP_x01
- removed SW2: RESET, SKRPACE010_C139797:SW_SKRPACE010_C139797, symbol Switch:SW_Push
- removed SW3: POWER, Button_Switch_THT:SW_Slide_SPDT_Angled_CK_OS102011MA1Q, symbol Switch:SW_SPDT
- removed TS1: Touchscreen, FT6236_TOUCH_6P:FT6236_TOUCH_6P_ALIGNED_V3, symbol FT6236_TOUCH_6P:FT6236_TOUCH_6P
- removed U1: CH340C, Package_SO:SOIC-16_3.9x9.9mm_P1.27mm, symbol Interface_USB:CH340C
- removed U2: PCM5102, Package_SO:TSSOP-20_4.4x6.5mm_P0.65mm, symbol Audio:PCM5102
- removed U3: ES8388, Package_DFN_QFN:QFN-28-1EP_4x4mm_P0.45mm_EP2.6x2.6mm, symbol Audio:ES8388
- removed U4: ESP32-P4NRW32X, PCM_Espressif:ESP32-P4, symbol PCM_Espressif:ESP32-P4X
- removed U5, U7: TLV62569DBV, Package_TO_SOT_SMD:SOT-23-5, symbol Regulator_Switching:TLV62569DBV
- removed U6: W25Q256JVEIQ, Package_SO:SOIC-8_5.3x5.3mm_P1.27mm, symbol Memory_Flash:W25Q16JVSS
- removed U8: TPS61183RTJT, Package_TO_SOT_SMD:SOT-23-5, symbol Regulator_Linear:TPS7A20xxxDBV
- removed U9: ESP32-C6-MINI-1/U, PCM_Espressif:ESP32-C6-MINI-1, symbol PCM_Espressif:ESP32-C6-MINI-1/U
- removed Y1: 40Mhz, Crystal:Crystal_SMD_3225-4Pin_3.2x2.5mm, symbol Crystal_4Pin_GND24_KiCad10:Crystal_4Pin_GND24
- removed Y2: 32.768Khz, Crystal:Crystal_SMD_3215-2Pin_3.2x1.5mm, symbol Device:Crystal
- added BT1: BS-12-B3AA011, P4Local_Coin_Cell:MYOUNG_BS-12-B3AA011_C964729, symbol P4Symbol_Device:Battery_Cell
- added C1, C2: 220pF, P4Local_Capacitor_SMD:C_0603_1608Metric, symbol P4Symbol_Device:C
- added C10, C12, C136, C137, C14, C16, C17, C18, C19, C22, C23, C25, C29, C30, C33, C34, C5, C6, C65, C77, C82, C85, C86: 100nF, P4Local_Capacitor_SMD:C_0603_1608Metric, symbol P4Symbol_Device:C
- added C100, C135, C97, C98: 1uF, P4Core:C_0603_1608Metric, symbol P4_Core:C
- added C101, C115, C118: 100nF, P4Core:C_0402_1005Metric, symbol P4_Core:C
- added C102, C116, C99: 1uF, P4Core:C_0402_1005Metric, symbol P4_Core:C
- added C103, C104, C105, C107, C109, C110, C112, C114, C117, C127, C129, C131, C132, C133, C94, C95, C96: 100nF, P4Core:C_0603_1608Metric, symbol P4_Core:C
- added C106, C108, C111, C113, C128, C134: 10uF, P4Core:C_0603_1608Metric, symbol P4_Core:C
- added C11, C13, C15, C21, C31, C32, C76, C9: 10uF, P4Local_Capacitor_SMD:C_0603_1608Metric, symbol P4Symbol_Device:C
- added C119, C120: 4.7uF, P4Core:C_0603_1608Metric, symbol P4_Core:C
- added C121, C130: 22uF, P4Core:C_0603_1608Metric, symbol P4_Core:C
- added C122, C123, C124, C125, C126: 22pF, P4Core:C_0603_1608Metric, symbol P4_Core:C
- added C138, C66, C81: 10uF, P4Local_Capacitor_SMD:C_0805_2012Metric, symbol P4Symbol_Device:C
- added C20, C88: 22uF, P4Local_Capacitor_SMD:C_0805_2012Metric, symbol P4Symbol_Device:C
- added C24, C26, C89: 2.2uF, P4Local_Capacitor_SMD:C_0603_1608Metric, symbol P4Symbol_Device:C
- added C27, C28: 2.2nF, P4Local_Capacitor_SMD:C_0603_1608Metric, symbol P4Symbol_Device:C
- added C3, C7: 100uF, P4Local_Capacitor_SMD:C_1206_3216Metric, symbol P4Symbol_Device:C_Polarized
- added C4: 4.7uF, P4Local_Capacitor_SMD:C_0603_1608Metric, symbol P4Symbol_Device:C
- added C75, C87, C90, C91: 1uF, P4Local_Capacitor_SMD:C_0603_1608Metric, symbol P4Symbol_Device:C
- added C92, C93: 100pF, P4Local_Capacitor_SMD:C_0603_1608Metric, symbol P4Symbol_Device:C
- added D1: Green LED, P4Local_LED_SMD:LED_0805_2012Metric, symbol P4Symbol_Device:LED
- added D3: SS34, P4Local_Diode_SMD:D_SMA, symbol P4Symbol_Device:D
- added DS1: FH34SRJ-40S-0.5SH(50), P4Local_Updated:ILI9488_40P_4inch_Checked, symbol P4Symbol_ILI9488_4IN_TFT_40P:ILI9488_4IN_TFT_40P
- added H1, H2, H3, H4: MountingHole, P4Local_MountingHole:MountingHole_3.2mm_M3, symbol P4Symbol_Mechanical:MountingHole
- added J1: TYPE-C-31-M-12, P4Local_Connector_USB:USB_C_Receptacle_HRO_TYPE-C-31-M-12, symbol P4Symbol_Connector:USB_C_Receptacle_USB2.0_16P
- added J10: S7B-PH-SM4-TB(LF)(SN), P4Local_Connector_JST:JST_PH_S7B-PH-SM4-TB_1x07-1MP_P2.00mm_Horizontal, symbol P4Symbol_Breakout:Breakout_J10
- added J11: S8B-PH-SM4-TB(LF)(SN), P4Local_Connector_JST:JST_PH_S8B-PH-SM4-TB_1x08-1MP_P2.00mm_Horizontal, symbol P4Symbol_Breakout:Breakout_J11
- added J12: S5B-PH-SM4-TB(LF)(SN), P4Local_Connector_JST:JST_PH_S5B-PH-SM4-TB_1x05-1MP_P2.00mm_Horizontal, symbol P4Symbol_Breakout:Breakout_J12
- added J13: S5B-PH-SM4-TB(LF)(SN), P4Local_Connector_JST:JST_PH_S5B-PH-SM4-TB_1x05-1MP_P2.00mm_Horizontal, symbol P4Symbol_Breakout:Breakout_J13
- added J2, J3: PJ-320D, P4Local_Connector_Audio_Han:HanElectricity_PJ320D_C22459515, symbol P4Symbol_PJ320D_KiCad10:AudioJack_PJ320D
- added J5: 67643-3911, P4Local_Connector_USB:USB_A_Molex_67643_Horizontal, symbol P4Symbol_Connector:USB_A
- added J6: DM3AT-SF-PEJM5, P4Local_Connector_Card:microSD_HC_Hirose_DM3AT-SF-PEJM5, symbol P4Symbol_Connector:Micro_SD_Card
- added J7: Conn_01x04_Pin, P4Local_Connector_PinHeader_2_54mm:PinHeader_1x04_P2.54mm_Vertical, symbol P4Symbol_Connector:Conn_01x04_Pin
- added J8: VBAT_SELECT, P4Local_Connector_JST:PinHeader_1x03_P2.54mm_Horizontal, symbol P4Symbol_Connector:Conn_01x03_Pin
- added J9: S5B-PH-SM4-TB(LF)(SN), P4Local_Connector_JST:JST_PH_S5B-PH-SM4-TB_1x05-1MP_P2.00mm_Horizontal, symbol P4Symbol_Breakout:Breakout_J9
- added L1: 600R@100MHz Ferrite, P4Local_Inductor_SMD:L_0603_1608Metric, symbol P4Symbol_Device:L_Ferrite
- added L2: 1uH, P4Core:L_INMICRO_IMTF201610, symbol P4_Core:L
- added Q2: AO3401A, P4Local_Package_TO_SOT_SMD:SOT-23, symbol P4Symbol_Transistor_FET:Q_PMOS_GSD
- added Q3: AO3400A, P4Local_Package_TO_SOT_SMD:SOT-23, symbol P4Symbol_Transistor_FET:Q_NMOS_GSD
- added Q4, Q5: S8050, P4Core:SOT-23, symbol P4_Core:S8050
- added R1, R2: 4.7k, P4Local_Resistor_SMD:R_0603_1608Metric, symbol P4Symbol_Device:R
- added R10, R11: 22R, P4Local_Resistor_SMD:R_0603_1608Metric, symbol P4Symbol_Device:R
- added R12, R18, R25, R29, R3, R30, R31, R32, R33, R34, R35, R36, R46, R61, R62, R9: 10k, P4Local_Resistor_SMD:R_0603_1608Metric, symbol P4Symbol_Device:R
- added R13, R14: 470R, P4Local_Resistor_SMD:R_0603_1608Metric, symbol P4Symbol_Device:R
- added R15: 100R, P4Local_Resistor_SMD:R_0603_1608Metric, symbol P4Symbol_Device:R
- added R16, R24, R27: 5.1k, P4Local_Resistor_SMD:R_0603_1608Metric, symbol P4Symbol_Device:R
- added R17, R5, R6, R7, R8: 33R, P4Local_Resistor_SMD:R_0603_1608Metric, symbol P4Symbol_Device:R
- added R23, R37: 100k, P4Local_Resistor_SMD:R_0603_1608Metric, symbol P4Symbol_Device:R
- added R26: 16R 0.5W, P4Local_Resistor_SMD:R_1210_3225Metric, symbol P4Symbol_Device:R
- added R4: 10R, P4Local_Resistor_SMD:R_0603_1608Metric, symbol P4Symbol_Device:R
- added R47: 1k, P4Local_Resistor_SMD:R_0603_1608Metric, symbol P4Symbol_Device:R
- added R48: 2k, P4Local_Resistor_SMD:R_0603_1608Metric, symbol P4Symbol_Device:R
- added R49, R50: 499k, P4Core:R_0603_1608Metric, symbol P4_Core:R
- added R51: 10M, P4Core:R_0603_1608Metric, symbol P4_Core:R
- added R52, R53: 10k, P4Core:R_0603_1608Metric, symbol P4_Core:R
- added R54, R55, R56, R57, R58, R59: 51k, P4Core:R_0603_1608Metric, symbol P4_Core:R
- added R60: 60.4k, P4Local_Resistor_SMD:R_0603_1608Metric, symbol P4Symbol_Device:R
- added SW1: EM-01KP, P4Local_Button_Switch_SMD:SW_DIP_SPSTx01_Slide_6.7x4.1mm_W8.61mm_P2.54mm_LowProfile, symbol P4Symbol_Switch:SW_DIP_x01
- added SW2: SKRPACE010, P4Local_SKRPACE010_C139797:SW_SKRPACE010_C139797, symbol P4Symbol_Switch:SW_Push
- added SW3: SK-12D02-G030, P4Local_Button_Switch_THT:SW_Slide_SPDT_Angled_CK_OS102011MA1Q, symbol P4Symbol_Switch:SW_SPDT
- added TS1: FH34SRJ-6S-0.5SH(50), P4Local_FT6236_TOUCH:Hirose_FH34SRJ-6S-0.5SH_FT6236, symbol P4Symbol_FT6236_TOUCH_6P:FT6236_TOUCH_6P
- added U1: ESP32-P4NRW32X, P4Core:ESP32-P4, symbol P4_Core:ESP32-P4X
- added U10: TPS2553DBVR, P4Core:SOT-23-6, symbol P4_Core:TPS2553DBVR
- added U2: PCM5102APWR, P4Local_Package_SO:TSSOP-20_4.4x6.5mm_P0.65mm, symbol P4Symbol_Audio:PCM5102
- added U3: ES8388, P4Local_Package_DFN_QFN:QFN-28-1EP_4x4mm_P0.45mm_EP2.6x2.6mm, symbol P4Symbol_Audio:ES8388
- added U4: CH340C, P4Local_Package_SO:SOIC-16_3.9x9.9mm_P1.27mm, symbol P4Symbol_Interface_USB:CH340C
- added U5: TLV62569DBVR, P4Core:SOT-23-5, symbol P4_Core:TLV62569DBV
- added U6: W25Q256JVEIQ, P4Core:WSON-8-1EP_8x6mm_P1.27mm_EP3.4x4.3mm, symbol P4_Core:W25Q16JVSS
- added U8: LD39150DT33-R, P4Local_Package_TO_SOT_SMD:TO-252-3_TabPin2, symbol P4Symbol_Regulator_Linear:LD39150DT33-R
- added U9: ESP32-C6-MINI-1-H4, P4Core:ESP32-C6-MINI-1, symbol P4_Core:ESP32-C6-MINI-1/U
- added Y1: 40Mhz, P4Core:Crystal_SMD_3225-4Pin_3.2x2.5mm, symbol P4_Core:Crystal_4Pin_GND24
- added Y2: 32.768Khz, P4Core:Crystal_SMD_3215-2Pin_3.2x1.5mm, symbol P4_Core:Crystal
Connections:
- net DTR: now also Q5.2 (E), R61.1, U4.13 (~{DTR})
- net EN_DCDC: now also U1.79 (EN_DCDC), U5.1 (EN)
- net ESP_EN: now also C75.1, J12.4 (ESP_EN), Q5.3 (C), R29.2, SW2.1, U1.103 (CHIP_PU)
- net ESP_LDO_VO1: now also C116.1, C127.2, C97.1, R52.1, U1.30 (VDD_FLASH_IO), U1.71 (VDDO_FLASH), U6.8 (VCC)
- net ESP_LDO_VO2: now also C101.1, C102.1, C98.1, U1.59 (VDD_PSRAM_0), U1.67 (VDD_PSRAM_1), U1.72 (VDDO_PSRAM)
- net ESP_LDO_VO3: now also C99.1, U1.73 (VDDO_3)
- net ESP_LDO_VO4: now also C100.1, C106.1, C107.1, U1.74 (VDDO_4), U1.85 (VDD_IO_5)
- net ESP_VDD_HP: now also C105.1, C113.1, C115.1, C121.1, C122.1, C128.1, C129.1, C130.1, C131.1, C94.1, L2.1, R50.1, U1.26 (VDD_HP_0), U1.54 (VDD_HP_1), U1.76 (VDD_HP_2), U1.91 (VDD_HP_3)
- net ES_DSDIN: now also R7.2, U3.6 (DSDIN)
- net ES_LRCK: now also R8.2, U3.7 (LRCK)
- net ES_MCLK: now also R17.2, U3.1 (MCLK)
- net ES_OUTL: now also R10.1, U3.12 (LOUT1)
- net ES_OUTR: now also R11.1, U3.11 (ROUT1)
- net FB_DCDC: now also C122.2, R49.1, R50.2, U1.78 (FB_DCDC), U5.5 (FB)
- net FLASH_CK_A: now also U1.32 (FLASH_CK), U6.6 (CLK)
- net FLASH_CS_A: now also R52.2, U1.27 (FLASH_CS), U6.1 (~{CS})
- net FLASH_D_A: now also U1.33 (FLASH_D), U6.5 (DI/IO_{0})
- net FLASH_HD_A: now also U1.31 (FLASH_HOLD), U6.7 (~{HOLD}/~{RESET}/IO_{3})
- net FLASH_Q_A: now also U1.28 (FLASH_Q), U6.2 (DO/IO_{1})
- net FLASH_WP_A: now also U1.29 (FLASH_WP), U6.3 (~{WP}/IO_{2})
- net GND: now also BT1.2 (-), C1.2, C10.2, C100.2, C101.2, C102.2, C103.2, C104.2, C105.2, C106.2, C107.2, C108.2, C109.2, C11.2, C110.2, C111.2, C112.2, C113.2, C114.2, C115.2, C116.2, C117.2, C118.2, C119.2, C12.2, C120.2, C121.2, C123.2, C124.2, C125.2, C126.2, C127.1, C128.2, C129.2, C13.2, C130.2, C131.2, C132.2, C133.2, C134.2, C135.2, C136.2, C137.2, C138.2, C14.2, C15.2, C16.2, C17.1, C18.1, C19.1, C2.2, C20.1, C21.2, C22.1, C23.1, C25.1, C26.1, C27.1, C28.1, C29.1, C30.1, C31.1, C32.2, C33.2, C34.1, C4.2, C5.2, C6.2, C65.2, C66.2, C75.2, C76.2, C77.2, C81.2, C82.2, C85.1, C86.2, C87.1, C88.1, C89.2, C9.2, C91.1, C92.2, C93.2, C94.2, C95.2, C96.2, C97.2, C98.2, C99.2, D1.1 (K), DS1.16 (GND), DS1.37 (GND), DS1.5 (GND), J1.A1 (GND), J1.A12 (GND), J1.B1 (GND), J1.B12 (GND), J1.SH (SHIELD), J10.1 (GND), J11.1 (GND), J12.1 (GND), J13.1 (GND), J2.R2 (Ring_2), J3.R2 (Ring_2), J3.S (Sleeve), J5.4 (GND), J5.SH (Shield), J6.6 (VSS), J6.9 (CD_A), J6.SH (SHIELD), J7.4 (Pin_4), J9.1 (GND), Q3.2 (S), R23.1, R24.2, R27.2, R37.1, R49.2, R60.1, SW2.2, TS1.6 (GND), U1.105 (GND), U10.2 (GND), U2.10 (DEMP), U2.11 (FLT), U2.12 (SCK), U2.16 (FMT), U2.19 (DGND), U2.3 (CPGND), U2.9 (AGND), U3.13 (HPGND), U3.18 (AGND), U3.29 (EPAD), U3.4 (DGND), U4.1 (GND), U5.2 (GND), U6.4 (GND), U8.2 (GND), U9.1 (GND), U9.11 (GND), U9.14 (GND), U9.2 (GND), U9.36 (GND), U9.37 (GND), U9.38 (GND), U9.39 (GND), U9.40 (GND), U9.41 (GND), U9.42 (GND), U9.43 (GND), U9.44 (GND), U9.45 (GND), U9.46 (GND), U9.47 (GND), U9.48 (GND), U9.49 (GND), U9.50 (GND), U9.51 (GND), U9.52 (GND), U9.53 (GND), Y1.2 (GND), Y1.4 (GND)
- net GPIO13: now also J11.4 (GPIO13), SW1.1, U1.14 (GPIO13)
- net GPIO2: now also J10.4 (GPIO2(SCK)), R15.1, U1.2 (GPIO2)
- net GPIO22: now also J11.5 (GPIO22), U1.24 (GPIO22/ADC1_CHANNEL6)
- net GPIO34: now also J11.6 (GPIO34), U1.65 (GPIO34)
- net GPIO53: now also Q2.1 (G), R36.2, R37.2, U1.97 (GPIO53/ADC2_CHANNEL4)
- net Headphone_L: now also C3.2, J2.T (Tip)
- net Headphone_R: now also C7.2, J2.R1 (Ring_1)
- net I2C_SCL: now also C2.1, J9.5 (GPIO8(SCL)), R1.2, TS1.3 (SCL), U1.8 (GPIO8), U3.28 (CCLK)
- net I2C_SDA: now also C1.1, J9.4 (GPIO7(SDA)), R2.2, TS1.2 (SDA), U1.7 (GPIO7), U3.27 (CDATA)
- net I2S_DSDIN: now also R7.1, U1.10 (GPIO9)
- net I2S_LRCK: now also R8.1, U1.11 (GPIO10)
- net I2S_MCLK: now also R17.1, U1.63 (GPIO32)
- net LED_K: now also DS1.34 (LED_K), DS1.35 (LED_K), DS1.36 (LED_K), Q3.3 (D)
- net Lineout_L: now also C27.2, J3.T (Tip), R13.2
- net Lineout_R: now also C28.2, J3.R1 (Ring_1), R14.2
- net PCM_DATA: now also U1.22 (GPIO20/ADC1_CHANNEL4), U2.14 (DIN)
- net PCM_LRCK: now also U1.25 (GPIO23/ADC1_CHANNEL7), U2.15 (LRCK)
- net RTS: now also Q4.2 (E), R62.1, U4.14 (~{RTS})
- net SD1_CLK: now also J6.5 (CLK), R33.2, U1.84 (GPIO43)
- net SD1_CMD: now also J6.3 (CMD), R32.2, U1.86 (GPIO44)
- net SD1_D0: now also J6.7 (DAT0), R34.2, U1.80 (GPIO39)
- net SD1_D1: now also J6.8 (DAT1), R46.2, U1.81 (GPIO40)
- net SD1_D2: now also J6.1 (DAT2), R30.2, U1.82 (GPIO41)
- net SD1_D3: now also J6.2 (DAT3/CD), R31.2, U1.83 (GPIO42)
- net TCH_INT: now also TS1.4 (INT), U1.89 (GPIO47)
- net TCH_RST: now also TS1.5 (RST), U1.64 (GPIO33)
- net TFT_CS: now also DS1.9 (CSX_SPI_CS), U1.95 (GPIO52/ADC2_CHANNEL3)
- net TFT_DC: now also DS1.10 (DCX_SPI_DC), U1.61 (GPIO31)
- net TFT_MISO: now also DS1.14 (SPI_MISO), U1.57 (GPIO28)
- net TFT_MOSI: now also DS1.13 (SPI_MOSI), U1.60 (GPIO30)
- net TFT_RESET: now also DS1.15 (RESET), U1.94 (GPIO51/ADC2_CHANNEL2)
- net TFT_SCK: now also DS1.11 (WRX_SPI_SCLK), U1.58 (GPIO29)
- net USBC_N: now also J1.A7 (D-), J1.B7 (D-), U4.6 (UD-)
- net USBC_P: now also J1.A6 (D+), J1.B6 (D+), U4.5 (UD+)
- net USB_5V: now also C65.1, C66.1, D3.2 (A), J10.2 (5V), J11.2 (5V), J12.2 (5V), J13.2 (5V), J9.2 (5V), R16.1, R26.1, SW3.2 (B), U8.1 (IN)
- net USB_N: now also J5.2 (D-), U1.55 (GPIO26/USB1P1_N1)
- net USB_P: now also J5.3 (D+), U1.56 (GPIO27/USB1P1_P1)
- net VBUS_5V: now also C136.1, C82.1, J1.A4 (VBUS), J1.A9 (VBUS), J1.B4 (VBUS), J1.B9 (VBUS), U10.1 (IN), U10.3 (EN)
- net XTAL_N: now also C124.1, U1.99 (XTAL_N), Y1.1 (XTAL1)
- net XTAL_P: now also C123.1, U1.100 (XTAL_P), Y1.3 (XTAL2)
- new net: D1.2 (A), R16.2
- new net: C3.1, R10.2
- new net: DS1.33 (LED_A), R26.2
- new net: C13.1, C14.1, U3.19 (ADCVREF)
- new net: D3.1 (K), J5.1 (VBUS)
- new net: R14.1, U2.7 (OUTR)
- new net: J6.10 (CD_B), R35.2, SW1.2
- new net: C10.1, C9.1, U3.10 (VREF)
- new net: C26.2, U2.5 (VNEG)
- new net: Q3.1 (G), R15.2, R23.2
- new net: C7.1, R11.2
- new net: R13.1, U2.6 (OUTL)
- new net: J1.A5 (CC1), R24.1
- new net: C15.1, C16.1, U3.20 (VMID)
- new net: J1.B5 (CC2), R27.1
- new net: C25.2, U2.18 (LDOO)
- new net: C24.1, U2.4 (CAPM)
- new net: C24.2, U2.2 (CAPP)
- new net: R12.2, U2.17 (XSMT)
- new net ADC_MIC_N: C91.2, C93.1, U3.23 (RIN1)
- new net ADC_MIC_P: C90.2, C92.1, U3.24 (LIN1)
- new net C6_BOOT: J7.1 (Pin_1), R9.1, U9.23 (GPIO9)
- new net C6_EN: C135.1, R53.2, U1.98 (GPIO54/ADC2_CHANNEL5), U9.8 (EN/CHIP_PU)
- new net C6_RX: J7.2 (Pin_2), U9.30 (U0RXD/GPIO17)
- new net C6_STRAP8: R18.1, U9.22 (GPIO8)
- new net C6_TX: J7.3 (Pin_3), U9.31 (U0TXD/GPIO16)
- new net COIN_CELL: BT1.1 (+), J8.1 (Pin_1)
- new net ES8388_3V3: C17.2, C32.1, C33.1, C34.2, C4.1, C5.1, C6.1, L1.2, R4.2, U3.16 (HPVDD), U3.2 (DVDD), U3.3 (PVDD)
- new net ESP_BOOT: J12.5 (ESP_BOOT), Q4.3 (C), R25.2, U1.66 (GPIO35)
- new net ES_ASDOUT: R5.2, U3.8 (ASDOUT)
- new net ES_AVDD: C11.1, C12.1, R4.1, R47.1, U3.17 (AVDD)
- new net ES_BCLK: R6.2, U3.5 (SCLK)
- new net GPIO3: J10.5 (GPIO3(MOSI)), U1.3 (GPIO3)
- new net GPIO4: J10.6 (GPIO4(MISO)), U1.4 (GPIO4)
- new net GPIO49: J11.7 (GPIO49), U1.92 (GPIO49/ADC2_CHANNEL0)
- new net GPIO5: J10.7 (GPIO5(CS)), U1.5 (GPIO5)
- new net GPIO50: J11.8 (GPIO50), U1.93 (GPIO50/ADC2_CHANNEL1)
- new net HEADSET_MIC: C90.1, J2.S (Sleeve), R48.2
- new net I2S_ASDOUT: R5.1, U1.12 (GPIO11)
- new net I2S_BCLK: R6.1, U1.13 (GPIO12)
- new net LDO_3V3: C103.1, C104.1, C108.1, C109.1, C110.1, C111.1, C112.1, C114.1, C117.1, C118.1, C119.1, C120.1, C132.1, C133.1, C134.1, C18.2, C19.2, C20.2, C21.1, C23.2, C29.2, C30.2, C81.1, C85.2, C87.2, C88.2, C95.1, C96.1, DS1.12 (RDX), DS1.38 (IM0), DS1.39 (IM1), DS1.40 (IM2), DS1.6 (VDDI), DS1.7 (VDD), J10.3 (3.3V), J11.3 (3.3V), J12.3 (3.3V), J13.3 (3.3V), J8.3 (Pin_3), J9.3 (3.3V), L1.1, Q2.2 (S), R1.1, R12.1, R18.2, R2.1, R25.1, R29.1, R3.2, R35.1, R36.1, R53.1, R54.1, R55.1, R56.1, R57.1, R58.1, R59.1, R9.2, TS1.1 (VDD), U1.101 (VDD_ANA), U1.21 (VDD_IO_0), U1.51 (VDD_USBPHY), U1.62 (VDD_IO_4), U1.75 (VDD_LDO), U1.77 (VDD_DCDCC), U1.9 (VDD_LP), U1.96 (VDD_IO_6), U2.1 (CPVDD), U2.20 (DVDD), U2.8 (AVDD), U3.26 (CE), U4.16 (VCC), U4.4 (V3), U5.4 (VIN), U8.3 (OUT), U9.3 (3V3)
- new net MIC_BIAS_FILTERED: C89.1, R47.2, R48.1
- new net P4_BOOT_BASE: Q4.1 (B), R61.2
- new net P4_C6_IO14: R58.2, U1.15 (GPIO14), U9.26 (GPIO20)
- new net P4_C6_IO15: R56.2, U1.16 (GPIO15), U9.27 (GPIO21)
- new net P4_C6_IO16: R55.2, U1.17 (GPIO16/ADC1_CHANNEL0), U9.28 (GPIO22)
- new net P4_C6_IO17: R54.2, U1.18 (GPIO17/ADC1_CHANNEL1), U9.29 (GPIO23)
- new net P4_C6_IO18: R57.2, U1.19 (GPIO18/ADC1_CHANNEL2), U9.25 (GPIO19)
- new net P4_C6_IO19: R59.2, U1.20 (GPIO19/ADC1_CHANNEL3), U9.24 (GPIO18)
- new net P4_C6_IO6: U1.6 (GPIO6), U9.5 (GPIO2/ADC1_CH2)
- new net P4_DCDC_SW: L2.2, U5.3 (SW)
- new net P4_EN_BASE: Q5.1 (B), R62.2
- new net P4_RTC0: C125.1, R51.1, U1.104 (GPIO0), Y2.1
- new net P4_RTC1: C126.1, R51.2, U1.1 (GPIO1), Y2.2
- new net P4_STRAP36: R3.1, U1.68 (GPIO36)
- new net PCM_BCLK: U1.23 (GPIO21/ADC1_CHANNEL5), U2.13 (BCK)
- new net SD_3V3: C76.1, C77.1, C86.1, J6.4 (VDD), Q2.3 (D), R30.1, R31.1, R32.1, R33.1, R34.1, R46.1
- new net U0RXD: J13.5 (U0RXD), U1.69 (GPIO37), U4.2 (TXD)
- new net U0TXD: J13.4 (U0TXD), U1.70 (GPIO38), U4.3 (RXD)
- new net USB_ILIM: R60.2, U10.5 (ILIM)
- new net USB_PROTECTED_5V: C137.1, C138.1, SW3.3 (C), U10.6 (OUT)
- new net VBAT: C22.2, C31.2, J8.2 (Pin_2), U1.102 (VDD_BAT)
- no-connect marks 64 -> 70
Other:
- note added: "32 MB QSPI flash"
- note added: "40 MHz / RTC crystals"
- note added: "5V USB-C COMPUTER INPUT PROTECTION TPS2553: IN from J1, OUT to SW3. Default limit <=500mA; R60 sets limit. Place U10 and C136/C137/C138/R60 together on side B beside J1."
- note added: "BT1: rechargeable VL1220 (12.5 x 2.0 mm), not CR1220. J8: one shunt only; 1-2 CELL, 2-3 3V3 / NO CELL. Charging requires verified firmware configuration and voltage; see revision notes."
- note added: "CTIA HEADSET: T=LEFT, R1=RIGHT, R2=GND, S=MIC/LINE INPUT"
- note added: "Core decoupling / oscillator loading / SDIO pull-ups"
- note added: "ESP32-C6-MINI — SDIO companion"
- note added: "ESP32-P4NRW32X — Waveshare GPIO mapping"
- note added: "JST-SH 2.0 mm BREAKOUTS — 3.3V LOGIC; 5V/3.3V PINS ARE POWER ONLY"
- note added: "Layout: place 100nF capacitors beside their supply pins; short ground return. Keep P4 regulator input/output/feedback loops short. Keep C6 antenna region free of copper and components on all layers."
- note added: "P4 / C6 CORE — separate ESP32-P4 + ESP32-C6-MINI"
- note added: "P4 AUTOMATIC DOWNLOAD / RESET — two Basic S8050 + 10k base resistors GPIO35: pull-up for normal boot; auto-program pulls low for download. GPIO36: 10k pull-up."
- note added: "P4 core regulator"
- note added: "P4 v3.x: populate both 499k feedback resistors and 22pF capacitor. Flash VCC, pull-up and VDD_FLASHIO supplied from VDDO_FLASH."
- note added: "RTC: primary CR2032; disable battery charging in firmware. J8 selects CELL or 3V3 for VDD_BAT. Never bridge all three pins."
